File: Devices/LedBar/PCB/0-10V.sch (KiCad schematic (older format))
At the start: 8 parts, among them J601 0-10V(1), U601 LM393

Commit message: Renamed libraries
Parts:
- J601: footprint AmbientLight:15EDGRC-3.5-2P -> RGBW-Bar:15EDGRC-3.5-2P
- TP601, TP602: footprint AmbientLight:TestPoint_Pad_D1.0mm -> RGBW-Bar:TestPoint_Pad_D1.0mm
Changed lines of the file:
@@
 F 0 "TP601" H 6708 4018 50  0000 L CNN
 F 1 "a_out" H 6708 3927 50  0000 L CNN
-F 2 "AmbientLight:TestPoint_Pad_D1.0mm" H 6850 3900 50  0001 C CNN
+F 2 "RGBW-Bar:TestPoint_Pad_D1.0mm" H 6850 3900 50  0001 C CNN
 F 3 "~" H 6850 3900 50  0001 C CNN
 	1    6650 3900
@@
 F 0 "J601" H 7880 4092 50  0000 L CNN
 F 1 "0-10V(1)" H 7880 4001 50  0000 L CNN
-F 2 "AmbientLight:15EDGRC-3.5-2P" H 7800 4100 50  0001 C CNN
+F 2 "RGBW-Bar:15EDGRC-3.5-2P" H 7800 4100 50  0001 C CNN
 F 3 "~" H 7800 4100 50  0001 C CNN
 	1    7800 4100
@@
 F 0 "TP602" H 8558 4518 50  0000 L CNN
 F 1 "gnd" H 8558 4427 50  0000 L CNN
-F 2 "AmbientLight:TestPoint_Pad_D1.0mm" H 8700 4400 50  0001 C CNN
+F 2 "RGBW-Bar:TestPoint_Pad_D1.0mm" H 8700 4400 50  0001 C CNN
 F 3 "~" H 8700 4400 50  0001 C CNN
 	1    8500 4400
