File: Devices/LedBar/PCB/Brown-out.sch (KiCad schematic (older format))
At the start: 13 parts, among them U601 LM393

Commit message: Renamed libraries
Parts:
- TP801: footprint AmbientLight:TestPoint_Pad_D1.0mm -> RGBW-Bar:TestPoint_Pad_D1.0mm
Changed lines of the file:
@@
 F 0 "TP801" H 5942 4526 50  0000 R CNN
 F 1 "BO" H 5942 4617 50  0000 R CNN
-F 2 "AmbientLight:TestPoint_Pad_D1.0mm" H 6200 4500 50  0001 C CNN
+F 2 "RGBW-Bar:TestPoint_Pad_D1.0mm" H 6200 4500 50  0001 C CNN
 F 3 "~" H 6200 4500 50  0001 C CNN
 	1    6000 4500
