File: Devices/LedBar/PCB/Rtc.sch (KiCad schematic (older format))
At the start: 4 parts, among them U901 DS1307Z+, Y901 23.768kHz

Commit message: Many small fixes
Parts:
- U901: I2C_Address (none) -> i2c: 0x68
Changed lines of the file:
@@
 F 2 "Package_SO:SOIC-8_3.9x4.9mm_P1.27mm" H 5500 3000 50  0001 C CNN
 F 3 "https://datasheets.maximintegrated.com/en/ds/DS1307.pdf" H 5500 3500 50  0001 C CNN
+F 4 "i2c: 0x68" H 5900 3150 50  0000 R CNN "I2C_Address"
 	1    5500 3500
 	1    0    0    -1
