File: Devices/LedBar/PCB/CenterBoard.sch (KiCad schematic (older format))
At the start: 6 parts, among them J1201 strip2_GRBW, J1202 Conn_02x06_Odd_Even, J1203 Strip3_GRBW, J1204 Strip2_GRB, J1205 Strip3_GRB

Commit message: Many small fixes
Parts:
- H1204: footprint MountingHole:MountingHole_3.2mm_M3 -> AmbientLight:MountingHole_3.2mm_Wall_0.8mm
Changed lines of the file:
@@
 Wire Wire Line
 	5150 4000 5150 4150
-Wire Wire Line
-	5750 3500 5850 3500
-Wire Wire Line
-	5750 3600 5850 3600
-Wire Wire Line
-	5750 3700 5850 3700
-Wire Wire Line
-	5750 3800 5850 3800
 Text Label 6050 3500 0    50   ~ 0
 strip3_w_out
@@
 F 0 "H1204" H 5400 3250 50  0000 L CNN
 F 1 "MountingHole" H 5250 3150 50  0000 L CNN
-F 2 "MountingHole:MountingHole_3.2mm_M3" H 5500 3000 50  0001 C CNN
+F 2 "AmbientLight:MountingHole_3.2mm_Wall_0.8mm" H 5500 3000 50  0001 C CNN
 F 3 "~" H 5500 3000 50  0001 C CNN
 	1    5500 3000
@@
 Wire Wire Line
 	6600 3900 7300 3900
-Connection ~ 5850 3600
 Wire Wire Line
-	5850 3600 6900 3600
-Connection ~ 5850 3500
+	5750 3500 7300 3500
 Wire Wire Line
-	5850 3500 7300 3500
-Connection ~ 5850 3800
+	5750 3600 6900 3600
 Wire Wire Line
-	5850 3800 6700 3800
-Connection ~ 5850 3700
+	5750 3700 6800 3700
 Wire Wire Line
-	5850 3700 6800 3700
+	5750 3800 6700 3800
 $EndSCHEMATC

Commit message: Renamed libraries
Parts:
- H1204: footprint AmbientLight:MountingHole_3.2mm_Wall_0.8mm -> RGBW-Bar:MountingHole_3.2mm_Wall_0.8mm
- J1201: footprint AmbientLight:GRBW-wire-solder-pads-R -> RGBW-Bar:GRBW-wire-solder-pads-R; symbol AmbientLight:Conn_GRBW -> RGBW-Bar:Conn_GRBW
- J1203: footprint AmbientLight:GRBW-wire-solder-pads-L -> RGBW-Bar:GRBW-wire-solder-pads-L; symbol AmbientLight:Conn_GRBW -> RGBW-Bar:Conn_GRBW
- J1204: footprint AmbientLight:GRB-wire-solder-pads-R -> RGBW-Bar:GRB-wire-solder-pads-R; symbol AmbientLight:Conn_GRB -> RGBW-Bar:Conn_GRB
- J1205: footprint AmbientLight:GRB-wire-solder-pads-L -> RGBW-Bar:GRB-wire-solder-pads-L; symbol AmbientLight:Conn_GRB -> RGBW-Bar:Conn_GRB
Changed lines of the file:
@@
 $EndDescr
 $Comp
-L AmbientLight:Conn_GRBW J?
+L RGBW-Bar:Conn_GRBW J?
 U 1 1 61892900
 P 7500 3700
@@
 F 0 "J1203" H 7400 3300 50  0000 L CNN
 F 1 "Strip3_GRBW" H 7250 3400 50  0000 L CNN
-F 2 "AmbientLight:GRBW-wire-solder-pads-L" H 7500 3700 50  0001 C CNN
+F 2 "RGBW-Bar:GRBW-wire-solder-pads-L" H 7500 3700 50  0001 C CNN
 F 3 "~" H 7500 3700 50  0001 C CNN
 	1    7500 3700
@@
 $EndComp
 $Comp
-L AmbientLight:Conn_GRBW J?
+L RGBW-Bar:Conn_GRBW J?
 U 1 1 6189334E
 P 3500 3700
@@
 F 0 "J1201" H 3418 3275 50  0000 C CNN
 F 1 "strip2_GRBW" H 3418 3366 50  0000 C CNN
-F 2 "AmbientLight:GRBW-wire-solder-pads-R" H 3500 3700 50  0001 C CNN
+F 2 "RGBW-Bar:GRBW-wire-solder-pads-R" H 3500 3700 50  0001 C CNN
 F 3 "~" H 3500 3700 50  0001 C CNN
 	1    3500 3700
@@
 F 0 "H1204" H 5400 3250 50  0000 L CNN
 F 1 "MountingHole" H 5250 3150 50  0000 L CNN
-F 2 "AmbientLight:MountingHole_3.2mm_Wall_0.8mm" H 5500 3000 50  0001 C CNN
+F 2 "RGBW-Bar:MountingHole_3.2mm_Wall_0.8mm" H 5500 3000 50  0001 C CNN
 F 3 "~" H 5500 3000 50  0001 C CNN
 	1    5500 3000
@@
 $EndComp
 $Comp
-L AmbientLight:Conn_GRB J?
+L RGBW-Bar:Conn_GRB J?
 U 1 1 618A2D3B
 P 3500 4850
@@
 F 0 "J1204" H 3418 4425 50  0000 C CNN
 F 1 "Strip2_GRB" H 3418 4516 50  0000 C CNN
-F 2 "AmbientLight:GRB-wire-solder-pads-R" H 3500 4850 50  0001 C CNN
+F 2 "RGBW-Bar:GRB-wire-solder-pads-R" H 3500 4850 50  0001 C CNN
 F 3 "~" H 3500 4850 50  0001 C CNN
 	1    3500 4850
@@
 	4100 3600 5250 3600
 $Comp
-L AmbientLight:Conn_GRB J?
+L RGBW-Bar:Conn_GRB J?
 U 1 1 618AC9EE
 P 7500 4850
@@
 F 0 "J1205" H 7400 4450 50  0000 L CNN
 F 1 "Strip3_GRB" H 7300 4550 50  0000 L CNN
-F 2 "AmbientLight:GRB-wire-solder-pads-L" H 7500 4850 50  0001 C CNN
+F 2 "RGBW-Bar:GRB-wire-solder-pads-L" H 7500 4850 50  0001 C CNN
 F 3 "~" H 7500 4850 50  0001 C CNN
 	1    7500 4850

Commit message: [Issue #001] Fix color channel order of strips
Parts:
- J1201: value strip2_GRBW -> strip2_RGBW; footprint RGBW-Bar:GRBW-wire-solder-pads-R -> RGBW-Bar:RGBW-wire-solder-pads-R; symbol RGBW-Bar:Conn_GRBW -> RGBW-Bar:Conn_RGBW
- J1203: value Strip3_GRBW -> Strip3_RGBW; footprint RGBW-Bar:GRBW-wire-solder-pads-L -> RGBW-Bar:RGBW-wire-solder-pads-L; symbol RGBW-Bar:Conn_GRBW -> RGBW-Bar:Conn_RGBW
- J1204: value Strip2_GRB -> Strip2_BRG; footprint RGBW-Bar:GRB-wire-solder-pads-R -> RGBW-Bar:BRG-wire-solder-pads-R; symbol RGBW-Bar:Conn_GRB -> RGBW-Bar:Conn_RGB
- J1205: value Strip3_GRB -> Strip3_BRG; footprint RGBW-Bar:GRB-wire-solder-pads-L -> RGBW-Bar:BRG-wire-solder-pads-L; symbol RGBW-Bar:Conn_GRB -> RGBW-Bar:Conn_RGB
Connections:
- net strip2_g_out: now also J1202.7 (Pin_7); no longer J1202.5 (Pin_5)
- net strip2_r_out: now also J1202.5 (Pin_5); no longer J1202.7 (Pin_7)
- net strip3_g_out: now also J1202.8 (Pin_8); no longer J1202.6 (Pin_6)
- net strip3_r_out: now also J1202.6 (Pin_6); no longer J1202.8 (Pin_8)
Changed lines of the file:
@@
 $EndDescr
 $Comp
-L RGBW-Bar:Conn_GRBW J?
+L RGBW-Bar:Conn_RGBW J?
 U 1 1 61892900
 P 7500 3700
@@
 AR Path="/6188050F/61892900" Ref="J1203"  Part="1"
 F 0 "J1203" H 7400 3300 50  0000 L CNN
-F 1 "Strip3_GRBW" H 7250 3400 50  0000 L CNN
-F 2 "RGBW-Bar:GRBW-wire-solder-pads-L" H 7500 3700 50  0001 C CNN
+F 1 "Strip3_RGBW" H 7250 3400 50  0000 L CNN
+F 2 "RGBW-Bar:RGBW-wire-solder-pads-L" H 7500 3700 50  0001 C CNN
 F 3 "~" H 7500 3700 50  0001 C CNN
 	1    7500 3700
@@
 $EndComp
 $Comp
-L RGBW-Bar:Conn_GRBW J?
+L RGBW-Bar:Conn_RGBW J?
 U 1 1 6189334E
 P 3500 3700
@@
 AR Path="/6188050F/6189334E" Ref="J1201"  Part="1"
 F 0 "J1201" H 3418 3275 50  0000 C CNN
-F 1 "strip2_GRBW" H 3418 3366 50  0000 C CNN
-F 2 "RGBW-Bar:GRBW-wire-solder-pads-R" H 3500 3700 50  0001 C CNN
+F 1 "strip2_RGBW" H 3418 3366 50  0000 C CNN
+F 2 "RGBW-Bar:RGBW-wire-solder-pads-R" H 3500 3700 50  0001 C CNN
 F 3 "~" H 3500 3700 50  0001 C CNN
 	1    3500 3700
@@
 Text Label 5000 3600 2    50   ~ 0
 strip2_b_out
+Text Label 5000 3800 2    50   ~ 0
+strip2_r_out
 Text Label 5000 3700 2    50   ~ 0
-strip2_r_out
-Text Label 5000 3800 2    50   ~ 0
 strip2_g_out
 Text Label 5000 3900 2    50   ~ 0
@@
 Text Label 6050 3600 0    50   ~ 0
 strip3_b_out
+Text Label 6050 3800 0    50   ~ 0
+strip3_r_out
 Text Label 6050 3700 0    50   ~ 0
-strip3_r_out
-Text Label 6050 3800 0    50   ~ 0
 strip3_g_out
 Text Label 6050 3900 0    50   ~ 0
@@
 $EndComp
 $Comp
-L RGBW-Bar:Conn_GRB J?
+L RGBW-Bar:Conn_RGB J?
 U 1 1 618A2D3B
 P 3500 4850
@@
 AR Path="/6188050F/618A2D3B" Ref="J1204"  Part="1"
 F 0 "J1204" H 3418 4425 50  0000 C CNN
-F 1 "Strip2_GRB" H 3418 4516 50  0000 C CNN
-F 2 "RGBW-Bar:GRB-wire-solder-pads-R" H 3500 4850 50  0001 C CNN
+F 1 "Strip2_BRG" H 3418 4516 50  0000 C CNN
+F 2 "RGBW-Bar:BRG-wire-solder-pads-R" H 3500 4850 50  0001 C CNN
 F 3 "~" H 3500 4850 50  0001 C CNN
 	1    3500 4850
@@
 	4100 3600 5250 3600
 $Comp
-L RGBW-Bar:Conn_GRB J?
+L RGBW-Bar:Conn_RGB J?
 U 1 1 618AC9EE
 P 7500 4850
@@
 AR Path="/6188050F/618AC9EE" Ref="J1205"  Part="1"
 F 0 "J1205" H 7400 4450 50  0000 L CNN
-F 1 "Strip3_GRB" H 7300 4550 50  0000 L CNN
-F 2 "RGBW-Bar:GRB-wire-solder-pads-L" H 7500 4850 50  0001 C CNN
+F 1 "Strip3_BRG" H 7300 4550 50  0000 L CNN
+F 2 "RGBW-Bar:BRG-wire-solder-pads-L" H 7500 4850 50  0001 C CNN
 F 3 "~" H 7500 4850 50  0001 C CNN
 	1    7500 4850
