File: Devices/LedBar/PCB/LedBar.kicad_pcb (KiCad board)
At the start: 2 copper layers, 63.5 x 99.3 mm, 163 parts, among them J1001 Conn_02x06_Odd_Even, J1002 Conn_02x06_Odd_Even, J1101 strip1_GRBW, J1102 Conn_01x05, J1103 Strip1_GRB, J1201 strip2_GRBW, J1202 Conn_02x06_Odd_Even, J1203 Strip3_GRBW, J1204 Strip2_GRB, J1205 Strip3_GRB, J1301 Conn_01x05, J1302 Strip4_GRBW, J1303 Strip4_GRB, J301 12VDC/5A, J401 RS485, J501 Left, J502 Center, J503 Right, J601 0-10V(1), J701 AVR-ISP-6, Q501 Si2302DS, Q502 Si2302DS, Q503 Si2302DS, Q504 Si2302DS, Q505 Si2302DS, Q506 Si2302DS, Q507 Si2302DS, Q508 Si2302DS, Q509 Si2302DS, Q510 Si2302DS, Q511 Si2302DS, Q512 Si2302DS, Q513 Si2302DS, Q514 Si2302DS, Q515 Si2302DS, Q516 Si2302DS, SW701 button, SW702 reset, SW703 SW_DIP_x05, U301 INA219AxD, U302 AMS1117-5.0, U401 ISO3082DW, U402 B0505S-1W-SIP4, U501 PCA9685PW, U601 LM393, U701 ATmega48PV-10AU-arduino, U901 DS1307Z+, Y701 14.7456Mhz, Y901 23.768kHz

Commit message: Many small fixes
Parts:
- H1102, H1204, H1301: footprint MountingHole:MountingHole_3.2mm_M3 -> AmbientLight:MountingHole_3.2mm_Wall_0.8mm
- H203: footprint MountingHole:MountingHole_4.3mm_M4 -> AmbientLight:MountingHole_4.3mm_M4_modified1
- turned H203 to 0 degrees
Other:
- board text added: "Created by: Roel Drost Revision: ${rev} (${rev_date}) https://github.com/Roel1983/RGBW-Bar"
- board text added: "MainBoard"
- board text added: "RGBW-Bar"
- board text removed: "C503/C505"
- board text removed: "Created by: Roel Drost Revision: ${rev} (${rev_date}) https://github.com/Roel1983/LEDBar2"
- board text removed: "F201"
- board text removed: "Fix test point (the footprint it self is on the wrong side)"
- board text removed: "LEDBar - MainBoard"
- board text removed: "M2"
- board text removed: "TODO: - Check other layers like Fab layers etc. - Fix swap FAB layer side of testpoints - Fix missing FAB layer of connectors - write functions to extract board layout and position/rotation of specific components -> export to SCAD variables include file - Make script to deploy the board, which will make sure the workspace is checked in, and the commit number and remote location are set. - check I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"
- board text removed: "U302"

Commit message: Renamed libraries
Parts:
- F301: footprint AmbientLight:Fuseholder_Cylinder-5x20mm_BLX_A_Horizontal -> RGBW-Bar:Fuseholder_Cylinder-5x20mm_BLX_A_Horizontal
- H1102, H1204, H1301: footprint AmbientLight:MountingHole_3.2mm_Wall_0.8mm -> RGBW-Bar:MountingHole_3.2mm_Wall_0.8mm
- H203: footprint AmbientLight:MountingHole_4.3mm_M4_modified1 -> RGBW-Bar:MountingHole_4.3mm_M4_modified1
- J1001: footprint AmbientLight:perpendicular_pcb_1mm_male_2x6 -> RGBW-Bar:perpendicular_pcb_1mm_male_2x6
- J1002: footprint AmbientLight:PinHeader_2x06_P200mm_PCB_edge -> RGBW-Bar:PinHeader_2x06_P200mm_PCB_edge
- J1101, J1201: footprint AmbientLight:GRBW-wire-solder-pads-R -> RGBW-Bar:GRBW-wire-solder-pads-R
- J1103, J1204: footprint AmbientLight:GRB-wire-solder-pads-R -> RGBW-Bar:GRB-wire-solder-pads-R
- J1203, J1302: footprint AmbientLight:GRBW-wire-solder-pads-L -> RGBW-Bar:GRBW-wire-solder-pads-L
- J1205, J1303: footprint AmbientLight:GRB-wire-solder-pads-L -> RGBW-Bar:GRB-wire-solder-pads-L
- J301: footprint AmbientLight:15EDGRC-3.81-2P -> RGBW-Bar:15EDGRC-3.81-2P
- J401: footprint AmbientLight:15EDGRC-3.5-3P -> RGBW-Bar:15EDGRC-3.5-3P
- J502: footprint AmbientLight:perpendicular_pcb_1mm_female_2x6 -> RGBW-Bar:perpendicular_pcb_1mm_female_2x6
- J601: footprint AmbientLight:15EDGRC-3.5-2P -> RGBW-Bar:15EDGRC-3.5-2P
- J701: footprint AmbientLight:ISP_P1.27mm_single_row -> RGBW-Bar:ISP_P1.27mm_single_row
- MB101, MB102, MB103, MB104, MB106: footprint AmbientLight:MouseBit -> RGBW-Bar:MouseBit
- MB105: footprint AmbientLight:MouseBit_modified1 -> RGBW-Bar:MouseBit_modified1
- TP301, TP302, TP303, TP304, TP401, TP402, TP403, TP404, TP405, TP406, TP407, TP408, TP409, TP501, TP502, TP503, TP504, TP601, TP602, TP701, TP702, TP703, TP704, TP705, TP706, TP707, TP708, TP709, TP710, TP711, TP712, TP801: footprint AmbientLight:TestPoint_Pad_D1.0mm -> RGBW-Bar:TestPoint_Pad_D1.0mm
- U402: footprint AmbientLight:B0505S-1W -> RGBW-Bar:B0505S-1W

Commit message: Added more vias
Routing:
- net GND_iso: vias 8 -> 9
- net GND: vias 99 -> 113

Commit message: Fixed microcontroller type
Parts:
- U701: value ATmega48PV-10AU-arduino -> ATmega328P-AU

Commit message: Released LedBar PCB v1.0
Other:
- board text added: "Created by: Roel Drost Revision: v1.0 (2022-06-26) https://github.com/Roel1983/RGBW-Bar"
- board text removed: "Created by: Roel Drost Revision: ${rev} (${rev_date}) https://github.com/Roel1983/RGBW-Bar"

Commit message: [Issue #001] Fix color channel order of strips
Parts:
- J1101: value strip1_GRBW -> strip1_RGBW; footprint RGBW-Bar:GRBW-wire-solder-pads-R -> RGBW-Bar:RGBW-wire-solder-pads-R
- J1103: value Strip1_GRB -> Strip1_BRG; footprint RGBW-Bar:GRB-wire-solder-pads-R -> RGBW-Bar:BRG-wire-solder-pads-R
- J1201: value strip2_GRBW -> strip2_RGBW; footprint RGBW-Bar:GRBW-wire-solder-pads-R -> RGBW-Bar:RGBW-wire-solder-pads-R
- J1203: value Strip3_GRBW -> Strip3_RGBW; footprint RGBW-Bar:GRBW-wire-solder-pads-L -> RGBW-Bar:RGBW-wire-solder-pads-L
- J1204: value Strip2_GRB -> Strip2_BRG; footprint RGBW-Bar:GRB-wire-solder-pads-R -> RGBW-Bar:BRG-wire-solder-pads-R
- J1205: value Strip3_GRB -> Strip3_BRG; footprint RGBW-Bar:GRB-wire-solder-pads-L -> RGBW-Bar:BRG-wire-solder-pads-L
- J1302: value Strip4_GRBW -> Strip4_RGBW; footprint RGBW-Bar:GRBW-wire-solder-pads-L -> RGBW-Bar:RGBW-wire-solder-pads-L
- J1303: value Strip4_GRB -> Strip4_BRG; footprint RGBW-Bar:GRB-wire-solder-pads-L -> RGBW-Bar:BRG-wire-solder-pads-L
- moved Q501 3.68 mm to (133.3, 111.5)
- moved Q502 3.68 mm to (143.8, 111.5)
- moved Q503 3.68 mm to (158.5, 111.5)
- moved Q504 3.68 mm to (168.9, 111.5)
- moved Q505 3.68 mm to (133.3, 107.8)
- moved Q506 3.68 mm to (143.8, 107.8)
- moved Q507 3.68 mm to (158.5, 107.8)
- moved Q508 3.68 mm to (168.9, 107.8)
- moved J1301 0.13 mm to (175.3, 51.8)
Connections:
- J1001 pad 5: /Perpendicular/strip3_g_out -> /Perpendicular/strip3_r_out
- J1001 pad 6: /Perpendicular/strip2_g_out -> /Perpendicular/strip2_r_out
- J1001 pad 7: /Perpendicular/strip3_r_out -> /Perpendicular/strip3_g_out
- J1001 pad 8: /Perpendicular/strip2_r_out -> /Perpendicular/strip2_g_out
- J1002 pad 5: /Perpendicular/strip3_g_out -> /Perpendicular/strip3_r_out
- J1002 pad 6: /Perpendicular/strip2_g_out -> /Perpendicular/strip2_r_out
- J1002 pad 7: /Perpendicular/strip3_r_out -> /Perpendicular/strip3_g_out
- J1002 pad 8: /Perpendicular/strip2_r_out -> /Perpendicular/strip2_g_out
- J1102 pad 2: /LeftBoard/strip1_g_out -> /LeftBoard/strip1_r_out
- J1102 pad 3: /LeftBoard/strip1_r_out -> /LeftBoard/strip1_g_out
- J1202 pad 5: /CenterBoard/strip2_g_out -> /CenterBoard/strip2_r_out
- J1202 pad 6: /CenterBoard/strip3_g_out -> /CenterBoard/strip3_r_out
- J1202 pad 7: /CenterBoard/strip2_r_out -> /CenterBoard/strip2_g_out
- J1202 pad 8: /CenterBoard/strip3_r_out -> /CenterBoard/strip3_g_out
- J1301 pad 3: /RightBoard/strip4_r_out -> /RightBoard/strip4_g_out
- J1301 pad 4: /RightBoard/strip4_g_out -> /RightBoard/strip4_r_out
- J501 pad 2: /Mainboard/Pca/strip1_g_out -> /Mainboard/Pca/strip1_r_out
- J501 pad 3: /Mainboard/Pca/strip1_r_out -> /Mainboard/Pca/strip1_g_out
- J502 pad 5: /Mainboard/Pca/strip3_g_out -> /Mainboard/Pca/strip3_r_out
- J502 pad 6: /Mainboard/Pca/strip2_g_out -> /Mainboard/Pca/strip2_r_out
- J502 pad 7: /Mainboard/Pca/strip3_r_out -> /Mainboard/Pca/strip3_g_out
- J502 pad 8: /Mainboard/Pca/strip2_r_out -> /Mainboard/Pca/strip2_g_out
- J503 pad 3: /Mainboard/Pca/strip4_r_out -> /Mainboard/Pca/strip4_g_out
- J503 pad 4: /Mainboard/Pca/strip4_g_out -> /Mainboard/Pca/strip4_r_out
Routing:
- net /RightBoard/strip4_r_out: track 16.8 -> 23.8 mm
- net /LeftBoard/strip1_r_out: track 18.5 -> 23.8 mm
- net /Mainboard/Pca/strip4_g: track 23.9 -> 19.5 mm, vias 2 -> 0
- net /Mainboard/Pca/strip3_g: track 14.5 -> 10.5 mm
- net /Mainboard/Pca/strip2_g: track 41.2 -> 37.2 mm, vias 2 -> 0
- net /Mainboard/Pca/strip1_g: track 38.8 -> 35.2 mm, vias 2 -> 0
- net /Mainboard/Pca/strip1_r: track 34.0 -> 37.6 mm
- net /Mainboard/Pca/strip4_r: track 18.8 -> 22.3 mm
- net /Mainboard/Pca/strip2_r: track 36.0 -> 39.5 mm
- net /Mainboard/Pca/strip3_r: track 11.0 -> 14.4 mm, vias 2 -> 0
- net /LeftBoard/strip1_g_out: track 18.1 -> 20.6 mm
- net /CenterBoard/strip3_g_out: track 19.6 -> 21.6 mm
- net /CenterBoard/strip2_g_out: track 19.6 -> 21.6 mm
- net /Mainboard/Pca/strip3_r_out: track 6.39 -> 8.32 mm
- net /Mainboard/Pca/strip3_g_out: track 8.32 -> 6.39 mm
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