File: Devices/LedBar/PCB/LedBar.kicad_pcb (KiCad board)
At the start: 2 copper layers, 63.5 x 99.3 mm, 163 parts, among them J1001 Conn_02x06_Odd_Even, J1002 Conn_02x06_Odd_Even, J1101 strip1_RGBW, J1102 Conn_01x05, J1103 Strip1_BRG, J1201 strip2_RGBW, J1202 Conn_02x06_Odd_Even, J1203 Strip3_RGBW, J1204 Strip2_BRG, J1205 Strip3_BRG, J1301 Conn_01x05, J1302 Strip4_RGBW, J1303 Strip4_BRG, J301 12VDC/5A, J401 RS485, J501 Left, J502 Center, J503 Right, J601 0-10V(1), J701 AVR-ISP-6, Q501 Si2302DS, Q502 Si2302DS, Q503 Si2302DS, Q504 Si2302DS, Q505 Si2302DS, Q506 Si2302DS, Q507 Si2302DS, Q508 Si2302DS, Q509 Si2302DS, Q510 Si2302DS, Q511 Si2302DS, Q512 Si2302DS, Q513 Si2302DS, Q514 Si2302DS, Q515 Si2302DS, Q516 Si2302DS, SW701 button, SW702 reset, SW703 SW_DIP_x05, U301 INA219AxD, U302 AMS1117-5.0, U401 ISO3082DW, U402 B0505S-1W-SIP4, U501 PCA9685PW, U601 LM393, U701 ATmega328P-AU, U901 DS1307Z+, Y701 14.7456Mhz, Y901 23.768kHz

Commit message: [Issue #005] Inverse brown-out LED
Parts:
- moved R703 0.13 mm to (130.7, 76.2)
Connections:
- D701 pad 1: GND -> Net-(D701-Pad1)
- D701 pad 2: Net-(D701-Pad2) -> +5V
- R703 pad 2: Net-(D701-Pad2) -> Net-(D701-Pad1)
Routing:
- net Net-(D701-Pad2): track 3.48 -> 0.00 mm
- net +5V: track 325.0 -> 328.4 mm
- net Net-(D701-Pad1): track 0.00 -> 2.78 mm
- net GND: track 446.7 -> 449.4 mm, vias 113 -> 116

Commit message: [Issue #013] Disable LED when at power up until initialization is complete
Parts:
- added D706: 1N4148, Diode_SMD:D_1206_3216Metric_Pad1.42x1.75mm_HandSolder, B.Cu at (125.0, 83.3)
- added R711: 10k, Resistor_SMD:R_0805_2012Metric_Pad1.20x1.40mm_HandSolder, B.Cu at (128.1, 82.9)
- TP704: value dbg1 -> ~pca_rdy~
- TP705: value dbg2 -> dbg1
- moved TP712 12.7 mm to (127.0, 96.5)
- moved R702 3.21 mm to (121.9, 83.1), turned to 90 degrees
- moved TP704 2.54 mm to (127.0, 91.4)
- moved TP705 2.54 mm to (127.0, 94.0)
- moved R703 0.51 mm to (130.7, 76.7)
- moved J701 0.44 mm to (122.3, 86.9)
Connections:
- TP704 pad 1: /Mainboard/Microcontroller/debug1 -> /Mainboard/Microcontroller/~pca_rdy~
- TP705 pad 1: /Mainboard/Microcontroller/debug2 -> /Mainboard/Microcontroller/debug1
- U701 pad 25: /Mainboard/Microcontroller/debug2 -> /Mainboard/Microcontroller/~pca_rdy~
Routing:
- net /Mainboard/Microcontroller/~pca_rdy~: track 0.00 -> 17.0 mm, vias 0 -> 2
- net /Mainboard/Pca/~oe~: track 49.6 -> 60.3 mm
- net GND: track 449.4 -> 457.7 mm, vias 116 -> 122
- net /Mainboard/Brown-out/~Brown_out~: track 85.5 -> 92.8 mm
- net +5V: track 328.4 -> 334.3 mm
- net /Mainboard/Microcontroller/~reset~: track 33.1 -> 37.2 mm
- net /Mainboard/Microcontroller/debug2: track 3.94 -> 0.00 mm
- net /Mainboard/Microcontroller/led3_mosi: track 48.4 -> 50.5 mm
- net /Mainboard/Microcontroller/led1_sck: track 61.9 -> 63.8 mm
- net /Mainboard/Microcontroller/led2_miso: track 52.2 -> 53.3 mm
- net /Mainboard/0-10V/a_in: track 116.4 -> 117.2 mm
- net /Mainboard/Microcontroller/debug1: track 5.53 -> 6.06 mm

Commit message: [Issue #016] Remove load resistor on +5V_iso
Parts:
- removed the R401 at (123.8, 124.1)
- moved TP405 3.59 mm to (121.9, 121.9)
- renumbered R402 to R401, R403 to R402
Routing:
- net GND_iso: vias 9 -> 10

Commit message: [Issue #004] Replace power connector for bigger connector
Parts:
- J301: footprint RGBW-Bar:15EDGRC-3.81-2P -> RGBW-Bar:2EDGRC-5.08-2P
- moved J301 0.79 mm to (169.7, 139.7)

Commit message: [Issue #008] Fix 5V power suppy so it doesn't fail dangerously
Parts:
- added D302: 5v1, Diode_SMD:D_1206_3216Metric_Pad1.42x1.75mm_HandSolder, B.Cu at (161.4, 124.9)
- added R304: 62R/0.25W, Resistor_SMD:R_1210_3225Metric_Pad1.30x2.65mm_HandSolder, B.Cu at (161.4, 127.8)
- moved D301 3.94 mm to (158.8, 134.2)
- moved C305 2.98 mm to (163.1, 133.3)
Connections:
- C305 pad 1: /Mainboard/Power/+12V_not_measured -> Net-(C305-Pad1)
- C306 pad 2: /Mainboard/Power/+12V_not_measured -> Net-(C305-Pad1)
- U302 pad 3: /Mainboard/Power/+12V_not_measured -> Net-(C305-Pad1)
Routing:
- net Net-(C305-Pad1): track 0.00 -> 9.68 mm
- net /Mainboard/Power/+12V_not_measured: track 33.9 -> 29.2 mm
- net GND: track 457.7 -> 456.5 mm
- net +5V: track 334.3 -> 334.9 mm

Commit message: [Issue #006] Fix shape of perpendicular board so it corresponds with width of J1002
Parts:
- moved MB104 1.52 mm to (152.4, 58.5)
Other:
- outline, holes or cut-outs redrawn

Commit message: [Issue #011] PCB: Make 'Left' and 'Right' board identical
Parts:
- J1102: footprint Connector_PinHeader_2.00mm:PinHeader_1x05_P2.00mm_Vertical -> RGBW-Bar:PinHeader_1x05_P2.00mm_Vertical_no_silk
- J1301: footprint Connector_PinHeader_2.00mm:PinHeader_1x05_P2.00mm_Vertical -> RGBW-Bar:PinHeader_1x05_P2.00mm_Vertical_no_silk; moved to F.Cu
- J1302: footprint RGBW-Bar:RGBW-wire-solder-pads-L -> RGBW-Bar:RGBW-wire-solder-pads-R
- J1303: footprint RGBW-Bar:BRG-wire-solder-pads-L -> RGBW-Bar:BRG-wire-solder-pads-R
- moved J1301 9.21 mm to (179.8, 59.8)
- moved J1302 5.59 mm to (174.8, 66.8)
- moved J1303 5.59 mm to (174.8, 54.8)
- moved H1301 4.57 mm to (179.8, 65.2), turned to 0 degrees
Connections:
- J1301 pad 1: /RightBoard/strip4_w_out -> /RightBoard/12V+
- J1301 pad 2: /RightBoard/strip4_b_out -> /RightBoard/strip4_r_out
- J1301 pad 4: /RightBoard/strip4_r_out -> /RightBoard/strip4_b_out
- J1301 pad 5: /RightBoard/12V+ -> /RightBoard/strip4_w_out
Other:
- board text removed: "Center"
