File: Devices/LedBar/PCB/Pca.sch (KiCad schematic (older format))
At the start: 29 parts, among them J501 Left, J502 Center, J503 Right, Q501 Si2302DS, Q502 Si2302DS, Q503 Si2302DS, Q504 Si2302DS, Q505 Si2302DS, Q506 Si2302DS, Q507 Si2302DS, Q508 Si2302DS, Q509 Si2302DS, Q510 Si2302DS, Q511 Si2302DS, Q512 Si2302DS, Q513 Si2302DS, Q514 Si2302DS, Q515 Si2302DS, Q516 Si2302DS, U501 PCA9685PW

Commit message: Many small fixes
Parts:
- U501: I2C_Address (none) -> i2c: 0x40
Changed lines of the file:
@@
 F 2 "Package_SO:TSSOP-28_4.4x9.7mm_P0.65mm" H 2525 1625 50  0001 L CNN
 F 3 "http://www.nxp.com/documents/data_sheet/PCA9685.pdf" H 2100 3300 50  0001 C CNN
+F 4 "i2c: 0x40" H 2500 2150 50  0000 C CNN "I2C_Address"
 	1    2500 2600
 	1    0    0    -1

Commit message: Renamed libraries
Parts:
- J502: footprint AmbientLight:perpendicular_pcb_1mm_female_2x6 -> RGBW-Bar:perpendicular_pcb_1mm_female_2x6
- TP501, TP502, TP503, TP504: footprint AmbientLight:TestPoint_Pad_D1.0mm -> RGBW-Bar:TestPoint_Pad_D1.0mm
Changed lines of the file:
@@
 F 0 "TP501" H 1442 2320 50  0000 R CNN
 F 1 "~pca_oe~" H 1442 2418 50  0000 R CNN
-F 2 "AmbientLight:TestPoint_Pad_D1.0mm" H 1700 2300 50  0001 C CNN
+F 2 "RGBW-Bar:TestPoint_Pad_D1.0mm" H 1700 2300 50  0001 C CNN
 F 3 "~" H 1700 2300 50  0001 C CNN
 	1    1500 2300
@@
 F 0 "J502" H 6100 5767 50  0000 C CNN
 F 1 "Center" H 6100 5676 50  0000 C CNN
-F 2 "AmbientLight:perpendicular_pcb_1mm_female_2x6" H 6050 5250 50  0001 C CNN
+F 2 "RGBW-Bar:perpendicular_pcb_1mm_female_2x6" H 6050 5250 50  0001 C CNN
 F 3 "~" H 6050 5250 50  0001 C CNN
 	1    6050 5250
@@
 F 0 "TP502" V 9150 1200 50  0000 R CNN
 F 1 "s1w" V 9300 1200 50  0000 R CNN
-F 2 "AmbientLight:TestPoint_Pad_D1.0mm" H 9450 1000 50  0001 C CNN
+F 2 "RGBW-Bar:TestPoint_Pad_D1.0mm" H 9450 1000 50  0001 C CNN
 F 3 "~" H 9450 1000 50  0001 C CNN
 	1    9250 1000
@@
 F 0 "TP504" V 10400 1000 50  0000 R CNN
 F 1 "s1w_o" V 10500 1000 50  0000 L CNN
-F 2 "AmbientLight:TestPoint_Pad_D1.0mm" H 10700 800 50  0001 C CNN
+F 2 "RGBW-Bar:TestPoint_Pad_D1.0mm" H 10700 800 50  0001 C CNN
 F 3 "~" H 10700 800 50  0001 C CNN
 	1    10500 800
@@
 F 0 "TP503" V 9900 1650 50  0000 R CNN
 F 1 "gnd" V 10000 1600 50  0000 R CNN
-F 2 "AmbientLight:TestPoint_Pad_D1.0mm" H 10200 1300 50  0001 C CNN
+F 2 "RGBW-Bar:TestPoint_Pad_D1.0mm" H 10200 1300 50  0001 C CNN
 F 3 "~" H 10200 1300 50  0001 C CNN
 	1    10000 1300

Commit message: [Issue #001] Fix color channel order of strips
Changed lines of the file:
@@
 Wire Wire Line
 	3250 5550 2700 5550
+Text Label 3200 5350 2    50   ~ 0
+strip1_g_out
 Text Label 3200 5250 2    50   ~ 0
-strip1_g_out
-Text Label 3200 5350 2    50   ~ 0
 strip1_r_out
 Text Label 3200 5450 2    50   ~ 0
@@
 Wire Wire Line
 	5750 5550 5000 5550
-Text Label 5050 5250 0    50   ~ 0
+Text Label 5050 5350 0    50   ~ 0
 strip2_g_out
 Text Label 3700 1900 2    50   ~ 0
 strip1_r
-Text Label 5050 5350 0    50   ~ 0
+Text Label 5050 5250 0    50   ~ 0
 strip2_r_out
 Text Label 5050 5450 0    50   ~ 0
@@
 	1    0    0    -1
 $EndComp
+Text Label 6950 5350 2    50   ~ 0
+strip3_g_out
 Text Label 6950 5250 2    50   ~ 0
-strip3_g_out
-Text Label 6950 5350 2    50   ~ 0
 strip3_r_out
 Text Label 6950 5450 2    50   ~ 0
@@
 Wire Wire Line
 	8750 5550 9300 5550
+Text Label 8800 5350 0    50   ~ 0
+strip4_g_out
 Text Label 8800 5250 0    50   ~ 0
-strip4_g_out
-Text Label 8800 5350 0    50   ~ 0
 strip4_r_out
 Text Label 8800 5450 0    50   ~ 0
