File: Devices/LedBar/PCB/Perpendicular.sch (KiCad schematic (older format))
At the start: 2 parts, among them J1001 Conn_02x06_Odd_Even, J1002 Conn_02x06_Odd_Even

Commit message: Renamed libraries
Parts:
- J1001: footprint AmbientLight:perpendicular_pcb_1mm_male_2x6 -> RGBW-Bar:perpendicular_pcb_1mm_male_2x6
- J1002: footprint AmbientLight:PinHeader_2x06_P200mm_PCB_edge -> RGBW-Bar:PinHeader_2x06_P200mm_PCB_edge
Changed lines of the file:
@@
 F 0 "J1001" H 6000 2917 50  0000 C CNN
 F 1 "Conn_02x06_Odd_Even" H 6000 2826 50  0000 C CNN
-F 2 "AmbientLight:perpendicular_pcb_1mm_male_2x6" H 5950 2500 50  0001 C CNN
+F 2 "RGBW-Bar:perpendicular_pcb_1mm_male_2x6" H 5950 2500 50  0001 C CNN
 F 3 "~" H 5950 2500 50  0001 C CNN
 	1    5950 2500
@@
 F 0 "J1002" H 6000 4867 50  0000 C CNN
 F 1 "Conn_02x06_Odd_Even" H 6000 4776 50  0000 C CNN
-F 2 "AmbientLight:PinHeader_2x06_P200mm_PCB_edge" H 5950 4450 50  0001 C CNN
+F 2 "RGBW-Bar:PinHeader_2x06_P200mm_PCB_edge" H 5950 4450 50  0001 C CNN
 F 3 "~" H 5950 4450 50  0001 C CNN
 	1    5950 4450

Commit message: [Issue #001] Fix color channel order of strips
Connections:
- net strip2_g_out: now also J1001.8 (Pin_8), J1002.8 (Pin_8); no longer J1001.6 (Pin_6), J1002.6 (Pin_6)
- net strip2_r_out: now also J1001.6 (Pin_6), J1002.6 (Pin_6); no longer J1001.8 (Pin_8), J1002.8 (Pin_8)
- net strip3_g_out: now also J1001.7 (Pin_7), J1002.7 (Pin_7); no longer J1001.5 (Pin_5), J1002.5 (Pin_5)
- net strip3_r_out: now also J1001.5 (Pin_5), J1002.5 (Pin_5); no longer J1001.7 (Pin_7), J1002.7 (Pin_7)
Changed lines of the file:
@@
 Text Label 5100 2400 0    50   ~ 0
 strip3_+12V_2
+Text Label 5100 2600 0    50   ~ 0
+strip3_g_out
 Text Label 5100 2500 0    50   ~ 0
-strip3_g_out
-Text Label 5100 2600 0    50   ~ 0
 strip3_r_out
 Text Label 5100 2700 0    50   ~ 0
@@
 Text Label 6300 2400 0    50   ~ 0
 strip2_+12V_2
+Text Label 6300 2600 0    50   ~ 0
+strip2_g_out
 Text Label 6300 2500 0    50   ~ 0
-strip2_g_out
-Text Label 6300 2600 0    50   ~ 0
 strip2_r_out
 Text Label 6300 2700 0    50   ~ 0
