File: Devices/LedBar/PCB/Microcontroller.sch (KiCad schematic (older format))
At the start: 44 parts, among them J701 AVR-ISP-6, SW701 button, SW702 reset, SW703 SW_DIP_x05, U701 ATmega48PV-10AU-arduino, Y701 14.7456Mhz

Commit message: Renamed libraries
Parts:
- J701: footprint AmbientLight:ISP_P1.27mm_single_row -> RGBW-Bar:ISP_P1.27mm_single_row
- TP701, TP702, TP703, TP704, TP705, TP706, TP707, TP708, TP709, TP710, TP711, TP712: footprint AmbientLight:TestPoint_Pad_D1.0mm -> RGBW-Bar:TestPoint_Pad_D1.0mm
- U701: symbol AmbientLight:ATmega48PV-10AU-arduino -> RGBW-Bar:ATmega48PV-10AU-arduino
Changed lines of the file:
@@
 $EndDescr
 $Comp
-L AmbientLight:ATmega48PV-10AU-arduino U701
+L RGBW-Bar:ATmega48PV-10AU-arduino U701
 U 1 1 608B13AD
 P 2500 3000
@@
 F 0 "J701" H 2120 6146 50  0000 R CNN
 F 1 "AVR-ISP-6" H 2120 6055 50  0000 R CNN
-F 2 "AmbientLight:ISP_P1.27mm_single_row" V 2200 6100 50  0001 C CNN
+F 2 "RGBW-Bar:ISP_P1.27mm_single_row" V 2200 6100 50  0001 C CNN
 F 3 " ~" H 1175 5500 50  0001 C CNN
 	1    2450 6050
@@
 F 0 "TP709" H 6942 2226 50  0000 R CNN
 F 1 "scl" H 6942 2317 50  0000 R CNN
-F 2 "AmbientLight:TestPoint_Pad_D1.0mm" H 7200 2200 50  0001 C CNN
+F 2 "RGBW-Bar:TestPoint_Pad_D1.0mm" H 7200 2200 50  0001 C CNN
 F 3 "~" H 7200 2200 50  0001 C CNN
 	1    7000 2200
@@
 F 0 "TP711" H 7442 2226 50  0000 R CNN
 F 1 "sda" H 7442 2317 50  0000 R CNN
-F 2 "AmbientLight:TestPoint_Pad_D1.0mm" H 7700 2200 50  0001 C CNN
+F 2 "RGBW-Bar:TestPoint_Pad_D1.0mm" H 7700 2200 50  0001 C CNN
 F 3 "~" H 7700 2200 50  0001 C CNN
 	1    7500 2200
@@
 F 0 "TP710" V 7048 3688 50  0000 L CNN
 F 1 "~reset~" V 7146 3688 50  0000 L CNN
-F 2 "AmbientLight:TestPoint_Pad_D1.0mm" H 7300 3500 50  0001 C CNN
+F 2 "RGBW-Bar:TestPoint_Pad_D1.0mm" H 7300 3500 50  0001 C CNN
 F 3 "~" H 7300 3500 50  0001 C CNN
 	1    7100 3500
@@
 F 0 "TP706" H 4542 6526 50  0000 R CNN
 F 1 "~button~" H 4542 6617 50  0000 R CNN
-F 2 "AmbientLight:TestPoint_Pad_D1.0mm" H 4800 6500 50  0001 C CNN
+F 2 "RGBW-Bar:TestPoint_Pad_D1.0mm" H 4800 6500 50  0001 C CNN
 F 3 "~" H 4800 6500 50  0001 C CNN
 	1    4600 6500
@@
 F 0 "TP704" V 4304 2988 50  0000 L CNN
 F 1 "dbg1" V 4395 2988 50  0000 L CNN
-F 2 "AmbientLight:TestPoint_Pad_D1.0mm" H 4550 2800 50  0001 C CNN
+F 2 "RGBW-Bar:TestPoint_Pad_D1.0mm" H 4550 2800 50  0001 C CNN
 F 3 "~" H 4550 2800 50  0001 C CNN
 	1    4350 2800
@@
 F 0 "TP705" V 4304 3288 50  0000 L CNN
 F 1 "dbg2" V 4395 3288 50  0000 L CNN
-F 2 "AmbientLight:TestPoint_Pad_D1.0mm" H 4550 3100 50  0001 C CNN
+F 2 "RGBW-Bar:TestPoint_Pad_D1.0mm" H 4550 3100 50  0001 C CNN
 F 3 "~" H 4550 3100 50  0001 C CNN
 	1    4350 3100
@@
 F 0 "TP707" H 4692 5076 50  0000 R CNN
 F 1 "gnd" H 4692 5167 50  0000 R CNN
-F 2 "AmbientLight:TestPoint_Pad_D1.0mm" H 4950 5050 50  0001 C CNN
+F 2 "RGBW-Bar:TestPoint_Pad_D1.0mm" H 4950 5050 50  0001 C CNN
 F 3 "~" H 4950 5050 50  0001 C CNN
 	1    4750 5050
@@
 F 0 "TP712" H 7942 3476 50  0000 R CNN
 F 1 "gnd" H 7942 3567 50  0000 R CNN
-F 2 "AmbientLight:TestPoint_Pad_D1.0mm" H 8200 3450 50  0001 C CNN
+F 2 "RGBW-Bar:TestPoint_Pad_D1.0mm" H 8200 3450 50  0001 C CNN
 F 3 "~" H 8200 3450 50  0001 C CNN
 	1    8000 3450
@@
 F 0 "TP703" H 4058 5168 50  0000 L CNN
 F 1 "a_in" H 4058 5077 50  0000 L CNN
-F 2 "AmbientLight:TestPoint_Pad_D1.0mm" H 4200 5050 50  0001 C CNN
+F 2 "RGBW-Bar:TestPoint_Pad_D1.0mm" H 4200 5050 50  0001 C CNN
 F 3 "~" H 4200 5050 50  0001 C CNN
 	1    4000 5050
@@
 F 0 "TP702" H 3558 5168 50  0000 L CNN
 F 1 "pwm" H 3558 5077 50  0000 L CNN
-F 2 "AmbientLight:TestPoint_Pad_D1.0mm" H 3700 5050 50  0001 C CNN
+F 2 "RGBW-Bar:TestPoint_Pad_D1.0mm" H 3700 5050 50  0001 C CNN
 F 3 "~" H 3700 5050 50  0001 C CNN
 	1    3500 5050
@@
 F 0 "TP701" H 2942 5076 50  0000 R CNN
 F 1 "gnd" H 2942 5167 50  0000 R CNN
-F 2 "AmbientLight:TestPoint_Pad_D1.0mm" H 3200 5050 50  0001 C CNN
+F 2 "RGBW-Bar:TestPoint_Pad_D1.0mm" H 3200 5050 50  0001 C CNN
 F 3 "~" H 3200 5050 50  0001 C CNN
 	1    3000 5050
@@
 F 0 "TP708" H 6142 2026 50  0000 R CNN
 F 1 "gnd" H 6142 2117 50  0000 R CNN
-F 2 "AmbientLight:TestPoint_Pad_D1.0mm" H 6400 2000 50  0001 C CNN
+F 2 "RGBW-Bar:TestPoint_Pad_D1.0mm" H 6400 2000 50  0001 C CNN
 F 3 "~" H 6400 2000 50  0001 C CNN
 	1    6200 2000

Commit message: Fixed microcontroller type
Parts:
- U701: value ATmega48PV-10AU-arduino -> ATmega328P-AU; symbol RGBW-Bar:ATmega48PV-10AU-arduino -> RGBW-Bar:ATmega328P-AU-arduino
Changed lines of the file:
@@
 $EndDescr
 $Comp
-L RGBW-Bar:ATmega48PV-10AU-arduino U701
+L RGBW-Bar:ATmega328P-AU-arduino U701
 U 1 1 608B13AD
 P 2500 3000
 F 0 "U701" H 3000 4450 50  0000 R CNN
-F 1 "ATmega48PV-10AU-arduino" V 1900 3000 50  0000 C CNN
+F 1 "ATmega328P-AU" V 1900 3000 50  0000 C CNN
 F 2 "Package_QFP:TQFP-32_7x7mm_P0.8mm" H 2450 3000 50  0001 C CIN
 F 3 "" H 2500 3000 50  0001 C CNN

Commit message: [Issue #005] Inverse brown-out LED
Other:
- moved on the sheet: D701
Changed lines of the file:
@@
 	4600 6600 4600 6750
-Wire Wire Line
-	6600 6650 6600 6850
 Wire Wire Line
 	6600 6150 6600 6350
@@
 F 3 "~" H 6600 6500 50  0001 C CNN
 	1    6600 6500
-	0    -1   -1   0
+	0    1    1    0
 $EndComp
 $Comp
@@
 $EndComp
 $Comp
-L power:GND #PWR0714
-U 1 1 619C9B0C
-P 6600 6850
-F 0 "#PWR0714" H 6600 6600 50  0001 C CNN
-F 1 "GND" H 6605 6677 50  0000 C CNN
-F 2 "" H 6600 6850 50  0001 C CNN
-F 3 "" H 6600 6850 50  0001 C CNN
-	1    6600 6850
-	1    0    0    -1
-$EndComp
-$Comp
 L Device:R R?
 U 1 1 619D14C8
@@
 Text Label 1600 6050 0    50   ~ 0
 led1_sck
+Wire Wire Line
+	6600 6650 6600 6850
+$Comp
+L power:+5V #PWR?
+U 1 1 636C480C
+P 6600 6850
+F 0 "#PWR?" H 6600 6700 50  0001 C CNN
+F 1 "+5V" H 6615 7023 50  0000 C CNN
+F 2 "" H 6600 6850 50  0001 C CNN
+F 3 "" H 6600 6850 50  0001 C CNN
+	1    6600 6850
+	-1   0    0    1
+$EndComp
 $EndSCHEMATC

Commit message: [Issue #013] Disable LED when at power up until initialization is complete
Parts:
- added D706: 1N4148, Diode_SMD:D_1206_3216Metric_Pad1.42x1.75mm_HandSolder, symbol Device:D
- added R711: 10k, Resistor_SMD:R_0805_2012Metric_Pad1.20x1.40mm_HandSolder, symbol Device:R
- TP704: value dbg1 -> ~pca_rdy~
- TP705: value dbg2 -> dbg1
Connections:
- net labels added: ~pca_rdy~
- net labels removed: debug2
- wire segments 130 -> 135
Other:
- moved on the sheet: TP705
Changed lines of the file:
@@
 Text Label 3500 2800 0    50   ~ 0
 debug1
-Text Label 3500 2900 0    50   ~ 0
-debug2
 Text HLabel 4000 3000 2    50   Output ~ 0
 tx_en
@@
 	3100 4200 4000 4200
 $Comp
-L Connector:TestPoint TP704
-U 1 1 609CDE03
+L Connector:TestPoint TP705
+U 1 1 609D0394
 P 4350 2800
-F 0 "TP704" V 4304 2988 50  0000 L CNN
+F 0 "TP705" V 4304 2988 50  0000 L CNN
 F 1 "dbg1" V 4395 2988 50  0000 L CNN
 F 2 "RGBW-Bar:TestPoint_Pad_D1.0mm" H 4550 2800 50  0001 C CNN
@@
 	0    1    1    0
 $EndComp
-$Comp
-L Connector:TestPoint TP705
-U 1 1 609D0394
-P 4350 3100
-F 0 "TP705" V 4304 3288 50  0000 L CNN
-F 1 "dbg2" V 4395 3288 50  0000 L CNN
-F 2 "RGBW-Bar:TestPoint_Pad_D1.0mm" H 4550 3100 50  0001 C CNN
-F 3 "~" H 4550 3100 50  0001 C CNN
-	1    4350 3100
-	0    1    1    0
-$EndComp
-Wire Wire Line
-	3100 2800 4350 2800
-Wire Wire Line
-	4350 3100 4350 2900
-Wire Wire Line
-	4350 2900 3100 2900
+Wire Wire Line
+	4000 2900 3100 2900
 Wire Wire Line
 	4750 2400 4750 2300
@@
 	-1   0    0    1
 $EndComp
-Text Label 3500 3700 0    50   ~ 0
-~pca_oe~
-Wire Wire Line
-	3100 3700 4000 3700
 Text Label 5900 5250 0    50   ~ 0
 ~pca_oe~
@@
 	6600 6650 6600 6850
 $Comp
-L power:+5V #PWR?
+L power:+5V #PWR0723
 U 1 1 636C480C
 P 6600 6850
-F 0 "#PWR?" H 6600 6700 50  0001 C CNN
+F 0 "#PWR0723" H 6600 6700 50  0001 C CNN
 F 1 "+5V" H 6615 7023 50  0000 C CNN
 F 2 "" H 6600 6850 50  0001 C CNN
@@
 	-1   0    0    1
 $EndComp
+$Comp
+L Device:D D706
+U 1 1 636E3AFB
+P 6600 5000
+F 0 "D706" V 6646 4920 50  0000 R CNN
+F 1 "1N4148" V 6555 4920 50  0000 R CNN
+F 2 "Diode_SMD:D_1206_3216Metric_Pad1.42x1.75mm_HandSolder" H 6600 5000 50  0001 C CNN
+F 3 "~" H 6600 5000 50  0001 C CNN
+	1    6600 5000
+	0    -1   -1   0
+$EndComp
+$Comp
+L Device:R R711
+U 1 1 636E6D37
+P 6600 4500
+F 0 "R711" H 6670 4546 50  0000 L CNN
+F 1 "10k" H 6670 4455 50  0000 L CNN
+F 2 "Resistor_SMD:R_0805_2012Metric_Pad1.20x1.40mm_HandSolder" V 6530 4500 50  0001 C CNN
+F 3 "~" H 6600 4500 50  0001 C CNN
+	1    6600 4500
+	1    0    0    -1
+$EndComp
+$Comp
+L power:+5V #PWR0714
+U 1 1 636E9562
+P 6600 4250
+F 0 "#PWR0714" H 6600 4100 50  0001 C CNN
+F 1 "+5V" H 6615 4423 50  0000 C CNN
+F 2 "" H 6600 4250 50  0001 C CNN
+F 3 "" H 6600 4250 50  0001 C CNN
+	1    6600 4250
+	1    0    0    -1
+$EndComp
+Wire Wire Line
+	6600 4250 6600 4350
+Wire Wire Line
+	6600 4650 6600 4750
+Wire Wire Line
+	6600 5150 6600 5250
+Wire Wire Line
+	6600 4750 5850 4750
+Connection ~ 6600 4750
+Wire Wire Line
+	6600 4750 6600 4850
+Text Label 5900 4750 0    50   ~ 0
+~pca_rdy~
+Text Label 5000 3600 0    50   ~ 0
+~pca_rdy~
+Text Label 3500 2900 0    50   ~ 0
+~pca_rdy~
+$Comp
+L Connector:TestPoint TP704
+U 1 1 63722A12
+P 6750 4750
+F 0 "TP704" V 6704 4938 50  0000 L CNN
+F 1 "~pca_rdy~" V 6795 4938 50  0000 L CNN
+F 2 "RGBW-Bar:TestPoint_Pad_D1.0mm" H 6950 4750 50  0001 C CNN
+F 3 "~" H 6950 4750 50  0001 C CNN
+	1    6750 4750
+	0    1    1    0
+$EndComp
+Wire Wire Line
+	6750 4750 6600 4750
+Wire Wire Line
+	3100 3700 4000 3700
+Text Label 3500 3700 0    50   ~ 0
+~pca_oe~
+Wire Wire Line
+	3100 2800 4350 2800
 $EndSCHEMATC
