File: Devices/LedBar/PCB/Power.sch (KiCad schematic (older format))
At the start: 20 parts, among them J301 12VDC/5A, U301 INA219AxD, U302 AMS1117-5.0

Commit message: Many small fixes
Parts:
- U301: I2C_Address (none) -> i2c: 0x44
Changed lines of the file:
@@
 F 2 "Package_SO:SOIC-8_3.9x4.9mm_P1.27mm" H 6800 1900 50  0001 C CNN
 F 3 "http://www.ti.com/lit/ds/symlink/ina219.pdf" H 6350 2150 50  0001 C CNN
+F 4 "i2c: 0x44" H 6000 2250 50  0000 C CNN "I2C_Address"
 	1    6000 2250
 	1    0    0    -1

Commit message: Renamed libraries
Parts:
- F301: footprint AmbientLight:Fuseholder_Cylinder-5x20mm_BLX_A_Horizontal -> RGBW-Bar:Fuseholder_Cylinder-5x20mm_BLX_A_Horizontal
- J301: footprint AmbientLight:15EDGRC-3.81-2P -> RGBW-Bar:15EDGRC-3.81-2P
- TP301, TP302, TP303, TP304: footprint AmbientLight:TestPoint_Pad_D1.0mm -> RGBW-Bar:TestPoint_Pad_D1.0mm
Changed lines of the file:
@@
 F 0 "F301" V 2553 4000 50  0000 C CNN
 F 1 "Max. 5A F" V 2644 4000 50  0000 C CNN
-F 2 "AmbientLight:Fuseholder_Cylinder-5x20mm_BLX_A_Horizontal" V 2680 4000 50  0001 C CNN
+F 2 "RGBW-Bar:Fuseholder_Cylinder-5x20mm_BLX_A_Horizontal" V 2680 4000 50  0001 C CNN
 F 3 "~" H 2750 4000 50  0001 C CNN
 	1    2750 4000
@@
 F 0 "J301" H 2150 4850 50  0000 C CNN
 F 1 "12VDC/5A" H 2250 4750 50  0000 R CNN
-F 2 "AmbientLight:15EDGRC-3.81-2P" H 2300 4850 50  0001 C CNN
+F 2 "RGBW-Bar:15EDGRC-3.81-2P" H 2300 4850 50  0001 C CNN
 F 3 "https://www.on-shore.com/wp-content/uploads/OSTOQXX3251.pdf" H 2300 4850 50  0001 C CNN
 	1    2300 4850
@@
 F 0 "TP301" V 5454 4188 50  0000 L CNN
 F 1 "+12V" V 5545 4188 50  0000 L CNN
-F 2 "AmbientLight:TestPoint_Pad_D1.0mm" H 5700 4000 50  0001 C CNN
+F 2 "RGBW-Bar:TestPoint_Pad_D1.0mm" H 5700 4000 50  0001 C CNN
 F 3 "~" H 5700 4000 50  0001 C CNN
 	1    5500 4000
@@
 F 0 "TP303" V 8954 4688 50  0000 L CNN
 F 1 "+5V" V 9045 4688 50  0000 L CNN
-F 2 "AmbientLight:TestPoint_Pad_D1.0mm" H 9200 4500 50  0001 C CNN
+F 2 "RGBW-Bar:TestPoint_Pad_D1.0mm" H 9200 4500 50  0001 C CNN
 F 3 "~" H 9200 4500 50  0001 C CNN
 	1    9000 4500
@@
 F 0 "TP304" H 8942 5626 50  0000 R CNN
 F 1 "gnd" H 8942 5717 50  0000 R CNN
-F 2 "AmbientLight:TestPoint_Pad_D1.0mm" H 9200 5600 50  0001 C CNN
+F 2 "RGBW-Bar:TestPoint_Pad_D1.0mm" H 9200 5600 50  0001 C CNN
 F 3 "~" H 9200 5600 50  0001 C CNN
 	1    9000 5600
@@
 F 0 "TP302" H 5942 5626 50  0000 R CNN
 F 1 "gnd" H 5942 5717 50  0000 R CNN
-F 2 "AmbientLight:TestPoint_Pad_D1.0mm" H 6200 5600 50  0001 C CNN
+F 2 "RGBW-Bar:TestPoint_Pad_D1.0mm" H 6200 5600 50  0001 C CNN
 F 3 "~" H 6200 5600 50  0001 C CNN
 	1    6000 5600

Commit message: [Issue #004] Replace power connector for bigger connector
Parts:
- J301: footprint RGBW-Bar:15EDGRC-3.81-2P -> RGBW-Bar:2EDGRC-5.08-2P
Changed lines of the file:
@@
 F 0 "J301" H 2150 4850 50  0000 C CNN
 F 1 "12VDC/5A" H 2250 4750 50  0000 R CNN
-F 2 "RGBW-Bar:15EDGRC-3.81-2P" H 2300 4850 50  0001 C CNN
-F 3 "https://www.on-shore.com/wp-content/uploads/OSTOQXX3251.pdf" H 2300 4850 50  0001 C CNN
+F 2 "RGBW-Bar:2EDGRC-5.08-2P" H 2300 4850 50  0001 C CNN
+F 3 "" H 2300 4850 50  0001 C CNN
 	1    2300 4850
 	1    0    0    1

Commit message: [Issue #008] Fix 5V power suppy so it doesn't fail dangerously
Parts:
- added D302: 5v1, Diode_SMD:D_1206_3216Metric_Pad1.42x1.75mm_HandSolder, symbol Device:D_Zener
- added R304: 62R/0.25W, Resistor_SMD:R_1210_3225Metric_Pad1.30x2.65mm_HandSolder, symbol Device:R
Connections:
- net +12V_not_measured: now also R304.2; no longer C305.1, C306.2, U302.3 (VI)
- net +5V: now also D302.1 (K)
- net GND: now also D302.2 (A)
- new net: C305.1, C306.2, R304.1, U302.3 (VI)
Changed lines of the file:
@@
 Wire Wire Line
 	2900 4000 3000 4000
-Wire Wire Line
-	5000 4000 5000 4600
 Connection ~ 5000 4000
 Wire Wire Line
 	5000 4900 5000 5500
-Wire Wire Line
-	4000 4600 4000 4500
 Wire Wire Line
 	4000 4900 4000 5500
@@
 	4350 3000 4350 3350
 Wire Wire Line
-	8000 4500 9000 4500
+	8000 4500 8500 4500
 Connection ~ 8000 4500
 Wire Wire Line
-	7500 5500 9000 5500
+	7500 5500 8500 5500
 Wire Wire Line
 	6000 2650 6000 3000
@@
 	6000 5500 6000 5600
 Wire Wire Line
-	4000 4500 6000 4500
-Connection ~ 4000 4500
-Wire Wire Line
-	4000 4500 4000 4000
-Connection ~ 6000 4500
-Wire Wire Line
 	5000 4000 5500 4000
 Connection ~ 5500 4000
@@
 Text Label 3100 4000 0    50   ~ 0
 +12V_not_measured
+Wire Wire Line
+	5000 4000 5000 4600
+Wire Wire Line
+	4000 4000 4000 4500
+$Comp
+L Device:R R304
+U 1 1 6381CA7A
+P 5500 4500
+F 0 "R304" V 5293 4500 50  0000 C CNN
+F 1 "62R/0.25W" V 5384 4500 50  0000 C CNN
+F 2 "Resistor_SMD:R_1210_3225Metric_Pad1.30x2.65mm_HandSolder" V 5430 4500 50  0001 C CNN
+F 3 "~" H 5500 4500 50  0001 C CNN
+	1    5500 4500
+	0    1    1    0
+$EndComp
+Wire Wire Line
+	4000 4500 5350 4500
+Connection ~ 4000 4500
+Wire Wire Line
+	4000 4500 4000 4600
+Wire Wire Line
+	5650 4500 6000 4500
+Connection ~ 6000 4500
+$Comp
+L power:PWR_FLAG #FLG0101
+U 1 1 638308BB
+P 6000 4500
+F 0 "#FLG0101" H 6000 4575 50  0001 C CNN
+F 1 "PWR_FLAG" H 6000 4673 50  0001 C CNN
+F 2 "" H 6000 4500 50  0001 C CNN
+F 3 "~" H 6000 4500 50  0001 C CNN
+	1    6000 4500
+	1    0    0    -1
+$EndComp
+$Comp
+L Device:D_Zener D302
+U 1 1 63837588
+P 8500 5000
+F 0 "D302" V 8454 5080 50  0000 L CNN
+F 1 "5v1" V 8545 5080 50  0000 L CNN
+F 2 "Diode_SMD:D_1206_3216Metric_Pad1.42x1.75mm_HandSolder" H 8500 5000 50  0001 C CNN
+F 3 "~" H 8500 5000 50  0001 C CNN
+	1    8500 5000
+	0    1    1    0
+$EndComp
+Wire Wire Line
+	8500 4850 8500 4500
+Connection ~ 8500 4500
+Wire Wire Line
+	8500 4500 9000 4500
+Wire Wire Line
+	8500 5150 8500 5500
+Connection ~ 8500 5500
+Wire Wire Line
+	8500 5500 9000 5500
 $EndSCHEMATC
