File: Devices/LedBar/PCB/LeftBoard.sch (KiCad schematic (older format))
At the start: 4 parts, among them J1101 strip1_GRBW, J1102 Conn_01x05, J1103 Strip1_GRB

Commit message: Many small fixes
Parts:
- H1102: footprint MountingHole:MountingHole_3.2mm_M3 -> AmbientLight:MountingHole_3.2mm_Wall_0.8mm
Changed lines of the file:
@@
 F 0 "H1102" H 6450 2750 50  0000 L CNN
 F 1 "MountingHole" H 6250 2650 50  0000 L CNN
-F 2 "MountingHole:MountingHole_3.2mm_M3" H 6500 2500 50  0001 C CNN
+F 2 "AmbientLight:MountingHole_3.2mm_Wall_0.8mm" H 6500 2500 50  0001 C CNN
 F 3 "~" H 6500 2500 50  0001 C CNN
 	1    6500 2500

Commit message: Renamed libraries
Parts:
- H1102: footprint AmbientLight:MountingHole_3.2mm_Wall_0.8mm -> RGBW-Bar:MountingHole_3.2mm_Wall_0.8mm
- J1101: footprint AmbientLight:GRBW-wire-solder-pads-R -> RGBW-Bar:GRBW-wire-solder-pads-R; symbol AmbientLight:Conn_GRBW -> RGBW-Bar:Conn_GRBW
- J1103: footprint AmbientLight:GRB-wire-solder-pads-R -> RGBW-Bar:GRB-wire-solder-pads-R; symbol AmbientLight:Conn_GRB -> RGBW-Bar:Conn_GRB
Changed lines of the file:
@@
 12V+
 $Comp
-L AmbientLight:Conn_GRBW J1101
+L RGBW-Bar:Conn_GRBW J1101
 U 1 1 618B5913
 P 4550 3250
@@
 F 0 "J1101" H 4468 2825 50  0000 C CNN
 F 1 "strip1_GRBW" H 4468 2916 50  0000 C CNN
-F 2 "AmbientLight:GRBW-wire-solder-pads-R" H 4550 3250 50  0001 C CNN
+F 2 "RGBW-Bar:GRBW-wire-solder-pads-R" H 4550 3250 50  0001 C CNN
 F 3 "~" H 4550 3250 50  0001 C CNN
 	1    4550 3250
@@
 	4750 3250 5250 3250
 $Comp
-L AmbientLight:Conn_GRB J1103
+L RGBW-Bar:Conn_GRB J1103
 U 1 1 618B591A
 P 4550 4400
@@
 F 0 "J1103" H 4468 3975 50  0000 C CNN
 F 1 "Strip1_GRB" H 4468 4066 50  0000 C CNN
-F 2 "AmbientLight:GRB-wire-solder-pads-R" H 4550 4400 50  0001 C CNN
+F 2 "RGBW-Bar:GRB-wire-solder-pads-R" H 4550 4400 50  0001 C CNN
 F 3 "~" H 4550 4400 50  0001 C CNN
 	1    4550 4400
@@
 F 0 "H1102" H 6450 2750 50  0000 L CNN
 F 1 "MountingHole" H 6250 2650 50  0000 L CNN
-F 2 "AmbientLight:MountingHole_3.2mm_Wall_0.8mm" H 6500 2500 50  0001 C CNN
+F 2 "RGBW-Bar:MountingHole_3.2mm_Wall_0.8mm" H 6500 2500 50  0001 C CNN
 F 3 "~" H 6500 2500 50  0001 C CNN
 	1    6500 2500

Commit message: [Issue #001] Fix color channel order of strips
Parts:
- J1101: value strip1_GRBW -> strip1_RGBW; footprint RGBW-Bar:GRBW-wire-solder-pads-R -> RGBW-Bar:RGBW-wire-solder-pads-R; symbol RGBW-Bar:Conn_GRBW -> RGBW-Bar:Conn_RGBW
- J1103: value Strip1_GRB -> Strip1_BRG; footprint RGBW-Bar:GRB-wire-solder-pads-R -> RGBW-Bar:BRG-wire-solder-pads-R; symbol RGBW-Bar:Conn_GRB -> RGBW-Bar:Conn_RGB
Connections:
- net strip1_g_out: now also J1102.3 (Pin_3); no longer J1102.2 (Pin_2)
- net strip1_r_out: now also J1102.2 (Pin_2); no longer J1102.3 (Pin_3)
Changed lines of the file:
@@
 Text Label 5500 3150 0    50   ~ 0
 strip1_b_out
+Text Label 5500 3350 0    50   ~ 0
+strip1_r_out
 Text Label 5500 3250 0    50   ~ 0
-strip1_r_out
-Text Label 5500 3350 0    50   ~ 0
 strip1_g_out
 Text Label 5500 3450 0    50   ~ 0
 12V+
 $Comp
-L RGBW-Bar:Conn_GRBW J1101
+L RGBW-Bar:Conn_RGBW J1101
 U 1 1 618B5913
 P 4550 3250
@@
 AR Path="/6188050F/618B5913" Ref="J?"  Part="1"
 F 0 "J1101" H 4468 2825 50  0000 C CNN
-F 1 "strip1_GRBW" H 4468 2916 50  0000 C CNN
-F 2 "RGBW-Bar:GRBW-wire-solder-pads-R" H 4550 3250 50  0001 C CNN
+F 1 "strip1_RGBW" H 4468 2916 50  0000 C CNN
+F 2 "RGBW-Bar:RGBW-wire-solder-pads-R" H 4550 3250 50  0001 C CNN
 F 3 "~" H 4550 3250 50  0001 C CNN
 	1    4550 3250
@@
 	4750 3250 5250 3250
 $Comp
-L RGBW-Bar:Conn_GRB J1103
+L RGBW-Bar:Conn_RGB J1103
 U 1 1 618B591A
 P 4550 4400
@@
 AR Path="/6188050F/618B591A" Ref="J?"  Part="1"
 F 0 "J1103" H 4468 3975 50  0000 C CNN
-F 1 "Strip1_GRB" H 4468 4066 50  0000 C CNN
-F 2 "RGBW-Bar:GRB-wire-solder-pads-R" H 4550 4400 50  0001 C CNN
+F 1 "Strip1_BRG" H 4468 4066 50  0000 C CNN
+F 2 "RGBW-Bar:BRG-wire-solder-pads-R" H 4550 4400 50  0001 C CNN
 F 3 "~" H 4550 4400 50  0001 C CNN
 	1    4550 4400

Commit message: [Issue #011] PCB: Make 'Left' and 'Right' board identical
Parts:
- J1102: footprint Connector_PinHeader_2.00mm:PinHeader_1x05_P2.00mm_Vertical -> RGBW-Bar:PinHeader_1x05_P2.00mm_Vertical_no_silk
Changed lines of the file:
@@
 F 0 "J1102" H 6418 2825 50  0000 C CNN
 F 1 "Conn_01x05" H 6418 2916 50  0000 C CNN
-F 2 "Connector_PinHeader_2.00mm:PinHeader_1x05_P2.00mm_Vertical" H 6500 3250 50  0001 C CNN
+F 2 "RGBW-Bar:PinHeader_1x05_P2.00mm_Vertical_no_silk" H 6500 3250 50  0001 C CNN
 F 3 "~" H 6500 3250 50  0001 C CNN
 	1    6500 3250
