File: Devices/LedBar/PCB/RightBoard.sch (KiCad schematic (older format))
At the start: 4 parts, among them J1301 Conn_01x05, J1302 Strip4_GRBW, J1303 Strip4_GRB

Commit message: Many small fixes
Parts:
- H1301: footprint MountingHole:MountingHole_3.2mm_M3 -> AmbientLight:MountingHole_3.2mm_Wall_0.8mm
Changed lines of the file:
@@
 F 0 "H1301" H 4450 2750 50  0000 L CNN
 F 1 "MountingHole" H 4250 2650 50  0000 L CNN
-F 2 "MountingHole:MountingHole_3.2mm_M3" H 4500 2500 50  0001 C CNN
+F 2 "AmbientLight:MountingHole_3.2mm_Wall_0.8mm" H 4500 2500 50  0001 C CNN
 F 3 "~" H 4500 2500 50  0001 C CNN
 	1    4500 2500

Commit message: Renamed libraries
Parts:
- H1301: footprint AmbientLight:MountingHole_3.2mm_Wall_0.8mm -> RGBW-Bar:MountingHole_3.2mm_Wall_0.8mm
- J1302: footprint AmbientLight:GRBW-wire-solder-pads-L -> RGBW-Bar:GRBW-wire-solder-pads-L; symbol AmbientLight:Conn_GRBW -> RGBW-Bar:Conn_GRBW
- J1303: footprint AmbientLight:GRB-wire-solder-pads-L -> RGBW-Bar:GRB-wire-solder-pads-L; symbol AmbientLight:Conn_GRB -> RGBW-Bar:Conn_GRB
Changed lines of the file:
@@
 $EndDescr
 $Comp
-L AmbientLight:Conn_GRBW J?
+L RGBW-Bar:Conn_GRBW J?
 U 1 1 618BFD61
 P 6450 3250
@@
 F 0 "J1302" H 6350 2850 50  0000 L CNN
 F 1 "Strip4_GRBW" H 6200 2950 50  0000 L CNN
-F 2 "AmbientLight:GRBW-wire-solder-pads-L" H 6450 3250 50  0001 C CNN
+F 2 "RGBW-Bar:GRBW-wire-solder-pads-L" H 6450 3250 50  0001 C CNN
 F 3 "~" H 6450 3250 50  0001 C CNN
 	1    6450 3250
@@
 $EndComp
 $Comp
-L AmbientLight:Conn_GRB J?
+L RGBW-Bar:Conn_GRB J?
 U 1 1 618BFD6C
 P 6450 4400
@@
 F 0 "J1303" H 6350 4000 50  0000 L CNN
 F 1 "Strip4_GRB" H 6250 4100 50  0000 L CNN
-F 2 "AmbientLight:GRB-wire-solder-pads-L" H 6450 4400 50  0001 C CNN
+F 2 "RGBW-Bar:GRB-wire-solder-pads-L" H 6450 4400 50  0001 C CNN
 F 3 "~" H 6450 4400 50  0001 C CNN
 	1    6450 4400
@@
 F 0 "H1301" H 4450 2750 50  0000 L CNN
 F 1 "MountingHole" H 4250 2650 50  0000 L CNN
-F 2 "AmbientLight:MountingHole_3.2mm_Wall_0.8mm" H 4500 2500 50  0001 C CNN
+F 2 "RGBW-Bar:MountingHole_3.2mm_Wall_0.8mm" H 4500 2500 50  0001 C CNN
 F 3 "~" H 4500 2500 50  0001 C CNN
 	1    4500 2500

Commit message: [Issue #001] Fix color channel order of strips
Parts:
- J1302: value Strip4_GRBW -> Strip4_RGBW; footprint RGBW-Bar:GRBW-wire-solder-pads-L -> RGBW-Bar:RGBW-wire-solder-pads-L; symbol RGBW-Bar:Conn_GRBW -> RGBW-Bar:Conn_RGBW
- J1303: value Strip4_GRB -> Strip4_BRG; footprint RGBW-Bar:GRB-wire-solder-pads-L -> RGBW-Bar:BRG-wire-solder-pads-L; symbol RGBW-Bar:Conn_GRB -> RGBW-Bar:Conn_RGB
Connections:
- net strip4_g_out: now also J1301.3 (Pin_3); no longer J1301.4 (Pin_4)
- net strip4_r_out: now also J1301.4 (Pin_4); no longer J1301.3 (Pin_3)
Changed lines of the file:
@@
 $EndDescr
 $Comp
-L RGBW-Bar:Conn_GRBW J?
+L RGBW-Bar:Conn_RGBW J?
 U 1 1 618BFD61
 P 6450 3250
@@
 AR Path="/6188050F/618BFD61" Ref="J?"  Part="1"
 F 0 "J1302" H 6350 2850 50  0000 L CNN
-F 1 "Strip4_GRBW" H 6200 2950 50  0000 L CNN
-F 2 "RGBW-Bar:GRBW-wire-solder-pads-L" H 6450 3250 50  0001 C CNN
+F 1 "Strip4_RGBW" H 6200 2950 50  0000 L CNN
+F 2 "RGBW-Bar:RGBW-wire-solder-pads-L" H 6450 3250 50  0001 C CNN
 F 3 "~" H 6450 3250 50  0001 C CNN
 	1    6450 3250
@@
 $EndComp
 $Comp
-L RGBW-Bar:Conn_GRB J?
+L RGBW-Bar:Conn_RGB J?
 U 1 1 618BFD6C
 P 6450 4400
@@
 AR Path="/6188055C/618BFD6C" Ref="J1303"  Part="1"
 F 0 "J1303" H 6350 4000 50  0000 L CNN
-F 1 "Strip4_GRB" H 6250 4100 50  0000 L CNN
-F 2 "RGBW-Bar:GRB-wire-solder-pads-L" H 6450 4400 50  0001 C CNN
+F 1 "Strip4_BRG" H 6250 4100 50  0000 L CNN
+F 2 "RGBW-Bar:BRG-wire-solder-pads-L" H 6450 4400 50  0001 C CNN
 F 3 "~" H 6450 4400 50  0001 C CNN
 	1    6450 4400
@@
 Text Label 5000 3450 0    50   ~ 0
 12V+
+Text Label 5000 3250 0    50   ~ 0
+strip4_g_out
 Text Label 5000 3350 0    50   ~ 0
-strip4_g_out
-Text Label 5000 3250 0    50   ~ 0
 strip4_r_out
 Text Label 5000 3150 0    50   ~ 0

Commit message: [Issue #011] PCB: Make 'Left' and 'Right' board identical
Parts:
- J1301: footprint Connector_PinHeader_2.00mm:PinHeader_1x05_P2.00mm_Vertical -> RGBW-Bar:PinHeader_1x05_P2.00mm_Vertical_no_silk
- J1302: footprint RGBW-Bar:RGBW-wire-solder-pads-L -> RGBW-Bar:RGBW-wire-solder-pads-R
- J1303: footprint RGBW-Bar:BRG-wire-solder-pads-L -> RGBW-Bar:BRG-wire-solder-pads-R
Connections:
- net 12V+: now also J1301.1 (Pin_1); no longer J1301.5 (Pin_5)
- net strip4_b_out: now also J1301.4 (Pin_4); no longer J1301.2 (Pin_2)
- net strip4_r_out: now also J1301.2 (Pin_2); no longer J1301.4 (Pin_4)
- net strip4_w_out: now also J1301.5 (Pin_5); no longer J1301.1 (Pin_1)
Changed lines of the file:
@@
 F 0 "J1302" H 6350 2850 50  0000 L CNN
 F 1 "Strip4_RGBW" H 6200 2950 50  0000 L CNN
-F 2 "RGBW-Bar:RGBW-wire-solder-pads-L" H 6450 3250 50  0001 C CNN
+F 2 "RGBW-Bar:RGBW-wire-solder-pads-R" H 6450 3250 50  0001 C CNN
 F 3 "~" H 6450 3250 50  0001 C CNN
 	1    6450 3250
@@
 F 0 "J1303" H 6350 4000 50  0000 L CNN
 F 1 "Strip4_BRG" H 6250 4100 50  0000 L CNN
-F 2 "RGBW-Bar:BRG-wire-solder-pads-L" H 6450 4400 50  0001 C CNN
+F 2 "RGBW-Bar:BRG-wire-solder-pads-R" H 6450 4400 50  0001 C CNN
 F 3 "~" H 6450 4400 50  0001 C CNN
 	1    6450 4400
@@
 AR Path="/618804D0/61891AC0" Ref="J?"  Part="1"
 AR Path="/6188055C/61891AC0" Ref="J1301"  Part="1"
-F 0 "J1301" H 4418 3667 50  0000 C CNN
-F 1 "Conn_01x05" H 4418 3576 50  0000 C CNN
-F 2 "Connector_PinHeader_2.00mm:PinHeader_1x05_P2.00mm_Vertical" H 4500 3250 50  0001 C CNN
+F 0 "J1301" H 4500 2850 50  0000 C CNN
+F 1 "Conn_01x05" H 4500 2950 50  0000 C CNN
+F 2 "RGBW-Bar:PinHeader_1x05_P2.00mm_Vertical_no_silk" H 4500 3250 50  0001 C CNN
 F 3 "~" H 4500 3250 50  0001 C CNN
 	1    4500 3250
-	-1   0    0    -1
+	-1   0    0    1
 $EndComp
 Connection ~ 5550 3450
