File: Devices/LedBar/PCB/Mainboard/Mainboard.kicad_pcb (KiCad board)
At the start: 2 copper layers, 63.5 x 73.7 mm, 144 parts, among them J301 12VDC/5A, J401 RS485, J501 Left, J502 Center, J503 Right, J601 0-10V(1), J701 AVR-ISP-6, Q501 Si2302DS, Q502 Si2302DS, Q503 Si2302DS, Q504 Si2302DS, Q505 Si2302DS, Q506 Si2302DS, Q507 Si2302DS, Q508 Si2302DS, Q509 Si2302DS, Q510 Si2302DS, Q511 Si2302DS, Q512 Si2302DS, Q513 Si2302DS, Q514 Si2302DS, Q515 Si2302DS, Q516 Si2302DS, SW701 button, SW702 reset, SW703 SW_DIP_x05, U301 INA219AxD, U302 AMS1117-5.0, U401 ISO3082DW, U402 B0505S-1W-SIP4, U501 PCA9685PW, U601 LM393, U701 ATmega328P-AU, U901 DS1307Z+, Y701 14.7456Mhz, Y901 23.768kHz

Commit message: [Issue #020] PCB: Serie resistors in RS485 bus must be 10R instead of 120R
Parts:
- R401, R402: value 120 -> 10R

Commit message: [Issue #023] PCB: Fix copper layer unprotected_12VDC
Routing:
- net /Power/unprotected_12VDC: track 67.9 -> 36.3 mm
- net GND: track 456.5 -> 460.2 mm, vias 122 -> 121
- net GND_iso: track 3.24 -> 2.12 mm
- net +5V: track 334.6 -> 335.3 mm
Other:
- net class 12V added: clearance 0.2, trace_width 1, via_dia 0.8, via_drill 0.4
- net class Default: trace_width 0.25 -> 0.2
- net class data added: clearance 0.2, trace_width 0.2, via_dia 0.8, via_drill 0.4
- net class gnd added: clearance 0.2, trace_width 0.25, via_dia 0.8, via_drill 0.4
- net class high_current added: clearance 0.2, trace_width 2.5, via_dia 0.8, via_drill 0.4
- net class high_current_unprotected added: clearance 0.5, trace_width 2.5, via_dia 0.8, via_drill 0.4
- net class low_current added: clearance 0.2, trace_width 0.35, via_dia 0.8, via_drill 0.4
- net class strip_out added: clearance 0.2, trace_width 0.5, via_dia 0.8, via_drill 0.4
