File: Devices/LedBar/PCB/Mainboard/0-10V.sch (KiCad schematic (older format))
At the start: 8 parts, among them J601 0-10V(1), U601 LM393

Commit message: [Issue #024] PCB: Optional PWM instead of 0-10v
Parts:
- added JP601: Jumper_3_Open, Jumper:SolderJumper-3_P1.3mm_Open_Pad1.0x1.5mm, symbol Jumper:Jumper_3_Open
Connections:
- wire segments 18 -> 24
Other:
- moved on the sheet: C601, J601, TP601, TP602
Changed lines of the file:
@@
 $Descr A4 11693 8268
 encoding utf-8
-Sheet 3 13
+Sheet 4 13
 Title "LedBar - MainBoard"
 Date "2022-06-26"
@@
 L Device:C C601
 U 1 1 608CAF7E
-P 6650 4250
-F 0 "C601" H 6765 4296 50  0000 L CNN
-F 1 "0.1uF" H 6765 4205 50  0000 L CNN
-F 2 "Capacitor_SMD:C_0805_2012Metric_Pad1.18x1.45mm_HandSolder" H 6688 4100 50  0001 C CNN
-F 3 "~" H 6650 4250 50  0001 C CNN
-	1    6650 4250
+P 7500 3750
+F 0 "C601" H 7615 3796 50  0000 L CNN
+F 1 "0.1uF" H 7615 3705 50  0000 L CNN
+F 2 "Capacitor_SMD:C_0805_2012Metric_Pad1.18x1.45mm_HandSolder" H 7538 3600 50  0001 C CNN
+F 3 "~" H 7500 3750 50  0001 C CNN
+	1    7500 3750
 	1    0    0    -1
 $EndComp
@@
 L power:GND #PWR0603
 U 1 1 608CB4E5
-P 6650 4500
-F 0 "#PWR0603" H 6650 4250 50  0001 C CNN
-F 1 "GND" H 6655 4327 50  0000 C CNN
-F 2 "" H 6650 4500 50  0001 C CNN
-F 3 "" H 6650 4500 50  0001 C CNN
-	1    6650 4500
-	1    0    0    -1
-$EndComp
-Wire Wire Line
-	6650 4500 6650 4400
-Wire Wire Line
-	6150 4000 6650 4000
-Wire Wire Line
-	6650 4000 6650 4100
+P 7500 4000
+F 0 "#PWR0603" H 7500 3750 50  0001 C CNN
+F 1 "GND" H 7505 3827 50  0000 C CNN
+F 2 "" H 7500 4000 50  0001 C CNN
+F 3 "" H 7500 4000 50  0001 C CNN
+	1    7500 4000
+	1    0    0    -1
+$EndComp
+Wire Wire Line
+	7500 4000 7500 3900
+Wire Wire Line
+	7500 3500 7500 3600
 $Comp
 L Connector:TestPoint TP601
 U 1 1 608CBD82
-P 6650 3900
-F 0 "TP601" H 6708 4018 50  0000 L CNN
-F 1 "a_out" H 6708 3927 50  0000 L CNN
-F 2 "RGBW-Bar:TestPoint_Pad_D1.0mm" H 6850 3900 50  0001 C CNN
-F 3 "~" H 6850 3900 50  0001 C CNN
-	1    6650 3900
-	1    0    0    -1
-$EndComp
-Wire Wire Line
-	6650 3900 6650 4000
-Connection ~ 6650 4000
+P 8000 3000
+F 0 "TP601" H 8058 3118 50  0000 L CNN
+F 1 "a_out" H 8058 3027 50  0000 L CNN
+F 2 "RGBW-Bar:TestPoint_Pad_D1.0mm" H 8200 3000 50  0001 C CNN
+F 3 "~" H 8200 3000 50  0001 C CNN
+	1    8000 3000
+	1    0    0    -1
+$EndComp
 $Comp
 L Connector_Generic:Conn_01x02 J601
 U 1 1 608CCE3C
-P 7800 4100
-F 0 "J601" H 7880 4092 50  0000 L CNN
-F 1 "0-10V(1)" H 7880 4001 50  0000 L CNN
-F 2 "RGBW-Bar:15EDGRC-3.5-2P" H 7800 4100 50  0001 C CNN
-F 3 "~" H 7800 4100 50  0001 C CNN
-	1    7800 4100
+P 8200 3600
+F 0 "J601" H 8280 3592 50  0000 L CNN
+F 1 "0-10V(1)" H 8280 3501 50  0000 L CNN
+F 2 "RGBW-Bar:15EDGRC-3.5-2P" H 8200 3600 50  0001 C CNN
+F 3 "~" H 8200 3600 50  0001 C CNN
+	1    8200 3600
 	1    0    0    1
 $EndComp
@@
 L power:GND #PWR0604
 U 1 1 608CDA6C
-P 7600 4600
-F 0 "#PWR0604" H 7600 4350 50  0001 C CNN
-F 1 "GND" H 7605 4427 50  0000 C CNN
-F 2 "" H 7600 4600 50  0001 C CNN
-F 3 "" H 7600 4600 50  0001 C CNN
-	1    7600 4600
-	1    0    0    -1
-$EndComp
-Wire Wire Line
-	7600 4600 7600 4100
+P 8000 4100
+F 0 "#PWR0604" H 8000 3850 50  0001 C CNN
+F 1 "GND" H 8005 3927 50  0000 C CNN
+F 2 "" H 8000 4100 50  0001 C CNN
+F 3 "" H 8000 4100 50  0001 C CNN
+	1    8000 4100
+	1    0    0    -1
+$EndComp
+Wire Wire Line
+	8000 4100 8000 3600
 $Comp
 L power:+12VA #PWR0601
@@
 $EndComp
 Wire Wire Line
-	6650 4000 7600 4000
-Wire Wire Line
-	4550 3900 5100 3900
+	4550 3900 5000 3900
 $Comp
 L Connector:TestPoint TP602
 U 1 1 61F20C57
-P 8500 4400
-F 0 "TP602" H 8558 4518 50  0000 L CNN
-F 1 "gnd" H 8558 4427 50  0000 L CNN
-F 2 "RGBW-Bar:TestPoint_Pad_D1.0mm" H 8700 4400 50  0001 C CNN
-F 3 "~" H 8700 4400 50  0001 C CNN
-	1    8500 4400
+P 8900 3900
+F 0 "TP602" H 8958 4018 50  0000 L CNN
+F 1 "gnd" H 8958 3927 50  0000 L CNN
+F 2 "RGBW-Bar:TestPoint_Pad_D1.0mm" H 9100 3900 50  0001 C CNN
+F 3 "~" H 9100 3900 50  0001 C CNN
+	1    8900 3900
 	1    0    0    -1
 $EndComp
@@
 L power:GND #PWR0605
 U 1 1 61F21EA9
-P 8500 4600
-F 0 "#PWR0605" H 8500 4350 50  0001 C CNN
-F 1 "GND" H 8505 4427 50  0000 C CNN
-F 2 "" H 8500 4600 50  0001 C CNN
-F 3 "" H 8500 4600 50  0001 C CNN
-	1    8500 4600
-	1    0    0    -1
-$EndComp
-Wire Wire Line
-	8500 4600 8500 4400
+P 8900 4100
+F 0 "#PWR0605" H 8900 3850 50  0001 C CNN
+F 1 "GND" H 8905 3927 50  0000 C CNN
+F 2 "" H 8900 4100 50  0001 C CNN
+F 3 "" H 8900 4100 50  0001 C CNN
+	1    8900 4100
+	1    0    0    -1
+$EndComp
+Wire Wire Line
+	8900 4100 8900 3900
+$Comp
+L Jumper:Jumper_3_Open JP601
+U 1 1 63879622
+P 7000 3500
+F 0 "JP601" V 7046 3587 50  0000 L CNN
+F 1 "Jumper_3_Open" V 6955 3587 50  0000 L CNN
+F 2 "Jumper:SolderJumper-3_P1.3mm_Open_Pad1.0x1.5mm" H 7000 3500 50  0001 C CNN
+F 3 "~" H 7000 3500 50  0001 C CNN
+	1    7000 3500
+	0    -1   1    0
+$EndComp
+Wire Wire Line
+	5000 3900 5000 3000
+Connection ~ 5000 3900
+Wire Wire Line
+	5000 3900 5100 3900
+Wire Wire Line
+	8000 3000 8000 3500
+Connection ~ 8000 3500
+Wire Wire Line
+	5000 3000 7000 3000
+Wire Wire Line
+	7000 3000 7000 3250
+Wire Wire Line
+	7000 3750 7000 4000
+Wire Wire Line
+	7000 4000 6150 4000
+Wire Wire Line
+	7150 3500 7500 3500
+Connection ~ 7500 3500
+Wire Wire Line
+	7500 3500 8000 3500
 $EndSCHEMATC
