File: Devices/LedBar/PCB/Mainboard/RS485.sch (KiCad schematic (older format))
At the start: 19 parts, among them J401 RS485, U401 ISO3082DW, U402 B0505S-1W-SIP4

Commit message: [Issue #020] PCB: Serie resistors in RS485 bus must be 10R instead of 120R
Parts:
- R401, R402: value 120 -> 10R
Changed lines of the file:
@@
 $Descr A4 11693 8268
 encoding utf-8
-Sheet 8 13
+Sheet 9 13
 Title "LedBar - MainBoard"
 Date "2022-06-26"
@@
 P 5850 4400
 F 0 "R401" V 6057 4400 50  0000 C CNN
-F 1 "120" V 5966 4400 50  0000 C CNN
+F 1 "10R" V 5966 4400 50  0000 C CNN
 F 2 "Resistor_SMD:R_0805_2012Metric_Pad1.20x1.40mm_HandSolder" V 5780 4400 50  0001 C CNN
 F 3 "~" H 5850 4400 50  0001 C CNN
@@
 P 5850 4600
 F 0 "R402" V 5650 4600 50  0000 C CNN
-F 1 "120" V 5750 4600 50  0000 C CNN
+F 1 "10R" V 5750 4600 50  0000 C CNN
 F 2 "Resistor_SMD:R_0805_2012Metric_Pad1.20x1.40mm_HandSolder" V 5780 4600 50  0001 C CNN
 F 3 "~" H 5850 4600 50  0001 C CNN
