File: Devices/LedBar/PCB/Mainboard/Microcontroller.sch (KiCad schematic (older format))
At the start: 46 parts, among them J701 AVR-ISP-6, SW701 button, SW702 reset, SW703 SW_DIP_x05, U701 ATmega328P-AU, Y701 14.7456Mhz

Commit message: [Issue #018] PCB: Devide PCB in different boards
Changed lines of the file:
@@
 $Descr A4 11693 8268
 encoding utf-8
-Sheet 7 13
+Sheet 6 13
 Title "LedBar - MainBoard"
 Date "2022-06-26"
@@
 AR Path="/608C0E66/619BE9CD" Ref="D?"  Part="1"
 AR Path="/6094F41A/619BE9CD" Ref="D?"  Part="1"
-AR Path="/608B1159/619BE9CD" Ref="D?"  Part="1"
+AR Path="/608B1159/619BE9CD" Ref="D701"  Part="1"
 AR Path="/617A8CB5/608B1159/619BE9CD" Ref="D701"  Part="1"
 F 0 "D701" V 6639 6382 50  0000 R CNN
@@
 AR Path="/608C0E66/619BE9D3" Ref="R?"  Part="1"
 AR Path="/6094F41A/619BE9D3" Ref="R?"  Part="1"
-AR Path="/608B1159/619BE9D3" Ref="R?"  Part="1"
+AR Path="/608B1159/619BE9D3" Ref="R703"  Part="1"
 AR Path="/617A8CB5/608B1159/619BE9D3" Ref="R703"  Part="1"
 F 0 "R703" H 6670 6046 50  0000 L CNN
@@
 P 3750 5200
 AR Path="/608C0E66/619D14C8" Ref="R?"  Part="1"
-AR Path="/608B1159/619D14C8" Ref="R?"  Part="1"
+AR Path="/608B1159/619D14C8" Ref="R701"  Part="1"
 AR Path="/617A8CB5/608B1159/619D14C8" Ref="R701"  Part="1"
 F 0 "R701" V 3543 5200 50  0000 C CNN
@@
 P 4000 5050
 AR Path="/608C0E66/61DFC26D" Ref="TP?"  Part="1"
-AR Path="/608B1159/61DFC26D" Ref="TP?"  Part="1"
+AR Path="/608B1159/61DFC26D" Ref="TP703"  Part="1"
 AR Path="/617A8CB5/608B1159/61DFC26D" Ref="TP703"  Part="1"
 F 0 "TP703" H 4058 5168 50  0000 L CNN
@@
 P 4000 5750
 AR Path="/608C0E66/61DFC274" Ref="#PWR?"  Part="1"
-AR Path="/608B1159/61DFC274" Ref="#PWR?"  Part="1"
+AR Path="/608B1159/61DFC274" Ref="#PWR0109"  Part="1"
 AR Path="/617A8CB5/608B1159/61DFC274" Ref="#PWR0709"  Part="1"
 F 0 "#PWR0709" H 4000 5500 50  0001 C CNN
@@
 P 4000 5400
 AR Path="/608C0E66/61DFC27A" Ref="C?"  Part="1"
-AR Path="/608B1159/61DFC27A" Ref="C?"  Part="1"
+AR Path="/608B1159/61DFC27A" Ref="C704"  Part="1"
 AR Path="/617A8CB5/608B1159/61DFC27A" Ref="C704"  Part="1"
 F 0 "C704" H 4115 5446 50  0000 L CNN
@@
 P 3500 5050
 AR Path="/608C0E66/619D14CE" Ref="TP?"  Part="1"
-AR Path="/608B1159/619D14CE" Ref="TP?"  Part="1"
+AR Path="/608B1159/619D14CE" Ref="TP702"  Part="1"
 AR Path="/617A8CB5/608B1159/619D14CE" Ref="TP702"  Part="1"
 F 0 "TP702" H 3558 5168 50  0000 L CNN
@@
 Text Label 5900 4750 0    50   ~ 0
 ~pca_rdy~
-Text Label 5000 3600 0    50   ~ 0
-~pca_rdy~
 Text Label 3500 2900 0    50   ~ 0

Commit message: Working on LEDs and Button for the Case
Parts:
- SW701: footprint Button_Switch_THT:SW_PUSH_6mm_H4.3mm -> Button_Switch_THT:SW_PUSH_6mm_H8mm
Changed lines of the file:
@@
 F 0 "SW701" V 4646 6902 50  0000 R CNN
 F 1 "button" V 4555 6902 50  0000 R CNN
-F 2 "Button_Switch_THT:SW_PUSH_6mm_H4.3mm" H 4600 7150 50  0001 C CNN
+F 2 "Button_Switch_THT:SW_PUSH_6mm_H8mm" H 4600 7150 50  0001 C CNN
 F 3 "~" H 4600 7150 50  0001 C CNN
 	1    4600 6950
