File: Devices/RS485-TTL/PCB/RS485-TTL.kicad_pcb (KiCad board)
At the start: 2 copper layers, 48.3 x 27.9 mm, 29 parts, among them J1 RS485, J2 Conn_01x05, U1 ISO3082DW, U2 B0505S-1W-SIP4

Commit message: Releasing RS485-TTL v1.0
Other:
- board text added: "Created by: Roel Drost Revision: v1.0 (2022-12-07) http://github.com/Roel1983.RGBW-Bar"
- board text removed: "Created by: Roel Drost Revision: v1.0 (2022-11-17) http://github.com/Roel1983.RGBW-Bar"
